File: _autosave-PD_Micro.kicad_sch (KiCad schematic)
At the start: 36 parts, among them J1 Conn_01x02, J2 Conn_01x02, J3 Conn_01x02, Q1 DMP3017SFK, Q2 DTC143E, U1 TPS62175DQC, U2 SRV05-4, U4 FUSB302BMPX

Commit message: librarys
Other:
- sheet Pico ports: added D+, D-, GND, VUSB; removed none
Changed lines of the file:
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@@
     (pin "6")
   )
-  (sheet (at 168.91 85.09) (size 16.51 7.62) (fields_autoplaced)
+  (sheet (at 168.91 85.09) (size 25.4 21.59) (fields_autoplaced)
     (stroke (width 0.1524) (type solid) (color 0 0 0 0))
     (fill (color 0 0 0 0.0000))
@@
       (effects (font (size 1.27 1.27)) (justify left bottom))
     )
-    (property "Sheet file" "USBC_PD.kicad_sch" (id 1) (at 168.91 93.2946 0)
+    (property "Sheet file" "USBC_PD.kicad_sch" (id 1) (at 168.91 107.2646 0)
       (effects (font (size 1.27 1.27)) (justify left top))
     )
+    (pin "D+" input (at 168.91 93.98 180)
+      (effects (font (size 1.27 1.27)) (justify left))
+    )
+    (pin "VUSB" input (at 168.91 87.63 180)
+      (effects (font (size 1.27 1.27)) (justify left))
+    )
+    (pin "GND" input (at 168.91 90.17 180)
+      (effects (font (size 1.27 1.27)) (justify left))
+    )
+    (pin "D-" input (at 168.91 96.52 180)
+      (effects (font (size 1.27 1.27)) (justify left))
+    )
   )
