File: PD_Micro.kicad_sch (KiCad schematic)
At the start: 36 parts, among them J1 Conn_01x02, J2 Conn_01x02, J3 Conn_01x02, Q1 DMP3017SFK, Q2 DTC143E, U1 TPS62175DQC, U2 SRV05-4, U4 FUSB302BMPX

Commit message: pico
Parts:
- added U?: Pico, RPi_Pico:RPi_Pico_SMD_TH, symbol MCU_RaspberryPi_and_Boards:Pico
Other:
- removed sheet Pico

Commit message: new pcb
Parts:
- added D2: WS2812B, LED_SMD:LED_WS2812B_PLCC4_5.0x5.0mm_P3.2mm, symbol LED:WS2812B
- C1, C2, C3, C4, C6, C7, C8: footprint -Passive:C_0805 -> Capacitor_SMD:C_0805_2012Metric
- C12, C13, C15, C16, C17: footprint -Passive:C_0603 -> Capacitor_SMD:C_0805_2012Metric
- R1, R11, R12, R2, R3, R4, R7, R8, R9: footprint -Passive:R_0603 -> Resistor_SMD:R_0805_2012Metric
- U3: renamed from U?; footprint RPi_Pico:RPi_Pico_SMD_TH -> MCU_RaspberryPi_and_Boards:RPi_Pico_SMD_TH
Connections:
- net +5V: now also U3.40 (VBUS), D2.1 (VDD)
- net GND: now also U3.13 (GND), U3.18 (GND), U3.23 (GND), U3.28 (GND), U3.3 (GND), U3.38 (GND), U3.42 (GND), U3.8 (GND), D2.3 (VSS)
- net at U3.1 (GPIO0): now also D2.4 (DIN)
Other:
- moved on the sheet: U3

Commit message: merge1
Parts:
- removed D1: SMF22A, -Discrete:D_SOD-123, symbol -Discrete:Diode_TVS
- removed J1, J2: Conn_01x02, -Connector:PinHeader_1x02_P2.54mm_Vertical, symbol -Connector:Conn_01x02
- removed J3: Conn_01x02, -Connector:TerminalBlock_3.5mm_2P, symbol -Connector:Conn_01x02
- added D?: SMF22A, -Discrete:D_SOD-123, symbol -Discrete:Diode_TVS
- added J? (x2): Conn_01x02, -Connector:PinHeader_1x02_P2.54mm_Vertical, symbol -Connector:Conn_01x02
- added J?: Conn_01x02, -Connector:TerminalBlock_3.5mm_2P, symbol -Connector:Conn_01x02
- added U?: oledSym, SSD1306:128x64OLED, symbol oled:oledSym
- added U?: ACS723xMATR-10AB, Package_SO:SOIC-16W_7.5x10.3mm_P1.27mm, symbol Sensor_Current:ACS723xMATR-10AB
Connections:
- net +5V: now also U?.1 (VCC), U?.10 (VCC)
- net D10: now also U3.2 (GPIO1)
- net GND: now also D?.2 (A), J?.2 (Pin_2), J?.2 (Pin_2), J?.2 (Pin_2), U?.0 (GND), U?.13 (BW_SEL), U?.15 (GND)
- net OUT: now also D?.1 (K), J?.1 (Pin_1), J?.1 (Pin_1), J?.1 (Pin_1), U?.5 (IP-), U?.6 (IP-), U?.7 (IP-), U?.8 (IP-); no longer C4.1, Q1.4 (D), Q1.5 (D), Q1.6 (D)
- net SCL: now reaches U3.10 (GPIO7)
- net SCL: now also U?.2 (SCL)
- net ADC0: now reaches U3.31 (GPIO26_ADC0)
- net ADC0: now also U?.12 (VIOUT)
- net SDA: now reaches U3.9 (GPIO6)
- net SDA: now also U?.3 (SDA)
- new net: C4.1, Q1.4 (D), Q1.5 (D), Q1.6 (D), U?.1 (IP+), U?.2 (IP+), U?.3 (IP+), U?.4 (IP+)
Other:
- moved on the sheet: C1, C12, C13, C15, C16, C17, C2, C3, C4, C6, C7, C8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

Commit message: merge2
Parts:
- removed U?: oledSym, SSD1306:128x64OLED, symbol oled:oledSym
- added U6: oledSym, SSD1306:128x64OLED, symbol oled:oledSym
- gave numbers to parts that had none: 5
Connections:
- net +5V: now also U6.2 (VCC)
- net GND: now also U6.1 (GND)
- net SCL: now also U6.3 (SCL)
- net SDA: now also U6.4 (SDA)
Changed lines of the file:
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@@
   (symbol (lib_id "-Flag:GND") (at 58.42 39.37 270) (unit 1)
     (in_bom yes) (on_board yes) (fields_autoplaced)
-    (property "Reference" "#PWR?" (id 0) (at 52.07 39.37 0)
+    (property "Reference" "#PWR0108" (id 0) (at 52.07 39.37 0)
       (effects (font (size 1.27 1.27)) hide)
     )
@@
   (symbol (lib_id "-Flag:+5V") (at 217.17 64.77 0) (unit 1)
     (in_bom yes) (on_board yes) (fields_autoplaced)
-    (property "Reference" "#PWR?" (id 0) (at 217.17 68.58 0)
+    (property "Reference" "#PWR0114" (id 0) (at 217.17 68.58 0)
       (effects (font (size 1.27 1.27)) hide)
     )
@@
   (symbol (lib_id "-Flag:GND") (at 35.56 25.4 90) (unit 1)
     (in_bom yes) (on_board yes)
-    (property "Reference" "#PWR?" (id 0) (at 41.91 25.4 0)
+    (property "Reference" "#PWR0110" (id 0) (at 41.91 25.4 0)
       (effects (font (size 1.27 1.27)) hide)
     )
@@
     (pin "1")
   )
-  (symbol (lib_id "oled:oledSym") (at 218.44 71.12 0) (unit 1)
-    (in_bom yes) (on_board yes) (fields_autoplaced)
-    (property "Reference" "U?" (id 0) (at 228.6 77.4699 0)
-      (effects (font (size 1.27 1.27)) (justify left))
-    )
-    (property "Value" "oledSym" (id 1) (at 228.6 80.0099 0)
-      (effects (font (size 1.27 1.27)) (justify left))
-    )
-    (property "Footprint" "SSD1306:128x64OLED" (id 2) (at 218.44 71.12 0)
-      (effects (font (size 1.27 1.27)) hide)
-    )
-    (property "Datasheet" "" (id 3) (at 218.44 71.12 0)
-      (effects (font (size 1.27 1.27)) hide)
-    )
-    (pin "0")
-    (pin "1")
-    (pin "2")
-    (pin "3")
-  )
   (symbol (lib_id "-Connector:Conn_01x02") (at 30.48 22.86 0) (mirror y) (unit 1)
     (in_bom yes) (on_board yes)
-    (property "Reference" "J?" (id 0) (at 28.448 23.0632 0)
+    (property "Reference" "J1" (id 0) (at 28.448 23.0632 0)
       (effects (font (size 1.27 1.27)) (justify left))
     )
@@
     (pin "1")
   )
+  (symbol (lib_name "oledSym_1") (lib_id "oled:oledSym") (at 218.44 71.12 0) (unit 1)
+    (in_bom yes) (on_board yes) (fields_autoplaced)
+    (property "Reference" "U6" (id 0) (at 228.6 77.4699 0)
+      (effects (font (size 1.27 1.27)) (justify left))
+    )
+    (property "Value" "oledSym" (id 1) (at 228.6 80.0099 0)
+      (effects (font (size 1.27 1.27)) (justify left))
+    )
+    (property "Footprint" "SSD1306:128x64OLED" (id 2) (at 218.44 71.12 0)
+      (effects (font (size 1.27 1.27)) hide)
+    )
+    (property "Datasheet" "" (id 3) (at 218.44 71.12 0)
+      (effects (font (size 1.27 1.27)) hide)
+    )
+    (pin "1")
+    (pin "2")
+    (pin "3")
+    (pin "4")
+  )
   (symbol (lib_id "-Flag:GND") (at 49.53 34.29 0) (unit 1)
     (in_bom yes) (on_board yes)
-    (property "Reference" "#PWR?" (id 0) (at 49.53 40.64 0)
+    (property "Reference" "#PWR0109" (id 0) (at 49.53 40.64 0)
       (effects (font (size 1.27 1.27)) hide)
     )
@@
   (symbol (lib_id "-Flag:GND") (at 35.56 34.29 90) (unit 1)
     (in_bom yes) (on_board yes)
-    (property "Reference" "#PWR?" (id 0) (at 41.91 34.29 0)
+    (property "Reference" "#PWR0111" (id 0) (at 41.91 34.29 0)
       (effects (font (size 1.27 1.27)) hide)
     )
@@
   (symbol (lib_id "-Discrete:Diode_TVS") (at 49.53 30.48 0) (unit 1)
     (in_bom yes) (on_board yes)
-    (property "Reference" "D?" (id 0) (at 51.2572 29.5148 0)
+    (property "Reference" "D1" (id 0) (at 51.2572 29.5148 0)
       (effects (font (size 1.27 1.27)) (justify left))
     )
@@
   (symbol (lib_id "Sensor_Current:ACS723xMATR-10AB") (at 71.12 39.37 270) (unit 1)
     (in_bom yes) (on_board yes) (fields_autoplaced)
-    (property "Reference" "U?" (id 0) (at 83.82 41.3894 0)
+    (property "Reference" "U5" (id 0) (at 83.82 41.3894 0)
       (effects (font (size 1.27 1.27)) (justify left))
     )
@@
   (symbol (lib_id "-Flag:GND") (at 205.74 68.58 0) (unit 1)
     (in_bom yes) (on_board yes) (fields_autoplaced)
-    (property "Reference" "#PWR?" (id 0) (at 205.74 74.93 0)
+    (property "Reference" "#PWR0113" (id 0) (at 205.74 74.93 0)
       (effects (font (size 1.27 1.27)) hide)
     )
@@
   (symbol (lib_id "-Flag:GND") (at 35.56 43.18 90) (unit 1)
     (in_bom yes) (on_board yes)
-    (property "Reference" "#PWR?" (id 0) (at 41.91 43.18 0)
+    (property "Reference" "#PWR0112" (id 0) (at 41.91 43.18 0)
       (effects (font (size 1.27 1.27)) hide)
     )
@@
   (symbol (lib_id "-Flag:+5V") (at 83.82 39.37 270) (unit 1)
     (in_bom yes) (on_board yes)
-    (property "Reference" "#PWR?" (id 0) (at 80.01 39.37 0)
+    (property "Reference" "#PWR0107" (id 0) (at 80.01 39.37 0)
       (effects (font (size 1.27 1.27)) hide)
     )
@@
   (symbol (lib_id "-Connector:Conn_01x02") (at 30.48 31.75 0) (mirror y) (unit 1)
     (in_bom yes) (on_board yes)
-    (property "Reference" "J?" (id 0) (at 28.448 31.9532 0)
+    (property "Reference" "J2" (id 0) (at 28.448 31.9532 0)
       (effects (font (size 1.27 1.27)) (justify left))
     )
@@
   (symbol (lib_id "-Connector:Conn_01x02") (at 30.48 40.64 0) (mirror y) (unit 1)
     (in_bom yes) (on_board yes)
-    (property "Reference" "J?" (id 0) (at 28.448 40.8432 0)
+    (property "Reference" "J3" (id 0) (at 28.448 40.8432 0)
       (effects (font (size 1.27 1.27)) (justify left))
     )
@@
       (reference "#PWR0106") (unit 1) (value "+5V") (footprint "")
     )
+    (path "/e302ed84-d962-4649-bcad-02fd87bbec8a"
+      (reference "#PWR0107") (unit 1) (value "+5V") (footprint "")
+    )
     (path "/06123694-435b-4ee6-ba53-4f08b14daa63"
-      (reference "#PWR?") (unit 1) (value "GND") (footprint "")
+      (reference "#PWR0108") (unit 1) (value "GND") (footprint "")
+    )
+    (path "/697c4e64-5ed4-4d71-9970-4090251582ae"
+      (reference "#PWR0109") (unit 1) (value "GND") (footprint "")
+    )
+    (path "/21044321-dcc0-41cc-b6b1-4cf7c7568f44"
+      (reference "#PWR0110") (unit 1) (value "GND") (footprint "")
+    )
+    (path "/6d89fbdd-2f48-4a39-92be-c6a8fe855ee7"
+      (reference "#PWR0111") (unit 1) (value "GND") (footprint "")
+    )
+    (path "/dbe99452-b83e-44fd-b094-83f289422357"
+      (reference "#PWR0112") (unit 1) (value "GND") (footprint "")
+    )
+    (path "/c7337224-ffd2-453e-b6ef-28d7acf99062"
+      (reference "#PWR0113") (unit 1) (value "GND") (footprint "")
     )
     (path "/1739b84f-a46b-4124-a614-91a1bde6b4cb"
-      (reference "#PWR?") (unit 1) (value "+5V") (footprint "")
-    )
-    (path "/21044321-dcc0-41cc-b6b1-4cf7c7568f44"
-      (reference "#PWR?") (unit 1) (value "GND") (footprint "")
-    )
-    (path "/697c4e64-5ed4-4d71-9970-4090251582ae"
-      (reference "#PWR?") (unit 1) (value "GND") (footprint "")
-    )
-    (path "/6d89fbdd-2f48-4a39-92be-c6a8fe855ee7"
-      (reference "#PWR?") (unit 1) (value "GND") (footprint "")
-    )
-    (path "/c7337224-ffd2-453e-b6ef-28d7acf99062"
-      (reference "#PWR?") (unit 1) (value "GND") (footprint "")
-    )
-    (path "/dbe99452-b83e-44fd-b094-83f289422357"
-      (reference "#PWR?") (unit 1) (value "GND") (footprint "")
-    )
-    (path "/e302ed84-d962-4649-bcad-02fd87bbec8a"
-      (reference "#PWR?") (unit 1) (value "+5V") (footprint "")
+      (reference "#PWR0114") (unit 1) (value "+5V") (footprint "")
     )
     (path "/00000000-0000-0000-0000-00005e821230"
@@
       (reference "C17") (unit 1) (value "330pF") (footprint "Capacitor_SMD:C_0805_2012Metric")
     )
+    (path "/82525001-5790-4411-8199-7402aa21c2bf"
+      (reference "D1") (unit 1) (value "SMF22A") (footprint "-Discrete:D_SOD-123")
+    )
     (path "/cb3e28a9-aa8e-44fc-8119-b84f843a551f"
       (reference "D2") (unit 1) (value "WS2812B") (footprint "LED_SMD:LED_WS2812B_PLCC4_5.0x5.0mm_P3.2mm")
     )
-    (path "/82525001-5790-4411-8199-7402aa21c2bf"
-      (reference "D?") (unit 1) (value "SMF22A") (footprint "-Discrete:D_SOD-123")
-    )
     (path "/00000000-0000-0000-0000-00005e5197fa"
       (reference "H1") (unit 1) (value "MountingHole") (footprint "-Hole:D1_8_PAD")
@@
     )
     (path "/3a984fd9-6cc5-448e-85c5-ba574e6e9774"
-      (reference "J?") (unit 1) (value "Conn_01x02") (footprint "-Connector:PinHeader_1x02_P2.54mm_Vertical")
+      (reference "J1") (unit 1) (value "Conn_01x02") (footprint "-Connector:PinHeader_1x02_P2.54mm_Vertical")
     )
     (path "/f9b2a6d5-58a1-4c93-9e1d-a7c57ddc2055"
-      (reference "J?") (unit 1) (value "Conn_01x02") (footprint "-Connector:PinHeader_1x02_P2.54mm_Vertical")
+      (reference "J2") (unit 1) (value "Conn_01x02") (footprint "-Connector:PinHeader_1x02_P2.54mm_Vertical")
     )
     (path "/ff797f7a-4157-4aa2-b5e9-5b2de39088c0"
-      (reference "J?") (unit 1) (value "Conn_01x02") (footprint "-Connector:TerminalBlock_3.5mm_2P")
+      (reference "J3") (unit 1) (value "Conn_01x02") (footprint "-Connector:TerminalBlock_3.5mm_2P")
     )
     (path "/00000000-0000-0000-0000-00005e7a6a70"
@@
       (reference "U4") (unit 1) (value "FUSB302BMPX") (footprint "-Chip:WQFN-14-1EP_2.5x2.5mm_P0.5mm_EP1.45x1.45mm")
     )
-    (path "/397bb19c-8324-4038-b251-8899d962435e"
-      (reference "U?") (unit 1) (value "oledSym") (footprint "SSD1306:128x64OLED")
-    )
     (path "/92d9bd57-2863-4e89-bab5-1b82f3694562"
-      (reference "U?") (unit 1) (value "ACS723xMATR-10AB") (footprint "Package_SO:SOIC-16W_7.5x10.3mm_P1.27mm")
+      (reference "U5") (unit 1) (value "ACS723xMATR-10AB") (footprint "Package_SO:SOIC-16W_7.5x10.3mm_P1.27mm")
+    )
+    (path "/663e4472-d7f6-444b-9a68-fef8d172256a"
+      (reference "U6") (unit 1) (value "oledSym") (footprint "SSD1306:128x64OLED")
     )
     (path "/00000000-0000-0000-0000-00005e65250b"
