File: PD_Micro.kicad_sch (KiCad schematic)
At the start: 61 parts, among them J1 Conn_01x02, J2 Conn_01x02, J3 Conn_01x02, J4 Conn_01x02, J5 Conn_01x02, Q1 DMP3017SFK, Q2 DTC143E, SW1 SW_DIP_x06, SW2 SW_DPST_x2, SW3 SW_Push, SW4 SW_Push, SW5 SW_DPST_x2, U1 SRV05-4, U2 Pico, U3 TPS62175DQC, U4 TPS62175DQC, U5 ACS723xLCTR-10AB, U6 oledSym

Commit message: v2.2
Parts:
- added R16: 10m, Capacitor_SMD:C_1206_3216Metric, symbol -Passive:R
- J1: footprint -Connector:TerminalBlock_3.5mm_2P -> TerminalBlock:TerminalBlock_bornier-2_P5.08mm
Connections:
- net +3.3V: now also U4.8 (~{SLEEP})
- net +5V: no longer U4.8 (~{SLEEP})
- net VBUS: now also R16.1; no longer U7.1 (ISENP), USB1.11 (VBUS), USB1.2 (VBUS)
- new net VDD: R16.2, U7.1 (ISENP), USB1.11 (VBUS), USB1.2 (VBUS)
- no-connect marks 2 -> 3
Changed lines of the file:
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@@
   (junction (at 181.61 130.81) (diameter 0) (color 0 0 0 0)
   )
+  (junction (at 185.42 80.01) (diameter 0) (color 0 0 0 0)
+  )
   (junction (at 240.03 41.91) (diameter 0) (color 0 0 0 0)
   )
@@
   (junction (at 251.46 41.91) (diameter 0) (color 0 0 0 0)
   )
-  (junction (at 185.42 80.01) (diameter 0) (color 0 0 0 0)
-  )
   (junction (at 92.71 102.87) (diameter 0) (color 0 0 0 0)
   )
@@
   (junction (at 49.53 22.86) (diameter 0) (color 0 0 0 0)
   )
+  (junction (at 185.42 87.63) (diameter 0) (color 0 0 0 0)
+  )
   (junction (at 154.94 43.18) (diameter 0) (color 0 0 0 0)
   )
@@
   )
   (no_connect (at 64.77 67.31))
+  (no_connect (at 104.14 147.32))
   (no_connect (at 64.77 82.55))
   (wire (pts (xy 243.84 41.91) (xy 251.46 41.91))
@@
     (stroke (width 0) (type default))
   )
-  (wire (pts (xy 251.46 41.91) (xy 269.24 41.91))
+  (wire (pts (xy 251.46 41.91) (xy 257.81 41.91))
     (stroke (width 0) (type default))
   )
@@
     (stroke (width 0) (type default))
   )
-  (wire (pts (xy 62.23 64.77) (xy 86.36 64.77))
+  (wire (pts (xy 62.23 64.77) (xy 66.04 64.77))
     (stroke (width 0) (type default))
   )
@@
     (stroke (width 0) (type default))
   )
-  (wire (pts (xy 185.42 87.63) (xy 185.42 80.01))
-    (stroke (width 0) (type default))
-  )
   (wire (pts (xy 199.39 123.19) (xy 200.66 123.19))
     (stroke (width 0) (type default))
@@
     (stroke (width 0) (type default))
   )
+  (wire (pts (xy 181.61 87.63) (xy 185.42 87.63))
+    (stroke (width 0) (type default))
+  )
   (wire (pts (xy 128.27 165.1) (xy 132.08 165.1))
     (stroke (width 0) (type default))
@@
     )
   )
-  (symbol (lib_id "-Flag:VBUS") (at 64.77 87.63 270) (mirror x) (unit 1)
-    (in_bom yes) (on_board yes) (dnp no)
-    (property "Reference" "#PWR030" (at 60.96 87.63 0)
-      (effects (font (size 1.27 1.27)) hide)
-    )
-    (property "Value" "VBUS" (at 67.31 87.63 90)
-      (effects (font (size 1.016 1.016)) (justify left))
-    )
-    (property "Footprint" "" (at 64.77 87.63 0)
-      (effects (font (size 1.27 1.27)) hide)
-    )
-    (property "Datasheet" "" (at 64.77 87.63 0)
-      (effects (font (size 1.27 1.27)) hide)
-    )
-    (pin "1")
-    (instances
-      (project "PD_Micro"
-        (path "/e63e39d7-6ac0-4ffd-8aa3-1841a4541b55"
-          (reference "#PWR030") (unit 1)
-        )
-      )
-    )
-  )
   (symbol (lib_id "-Passive:C") (at 66.04 97.79 0) (unit 1)
     (in_bom yes) (on_board yes) (dnp no)
@@
     )
   )
+  (symbol (lib_id "power:VDD") (at 181.61 87.63 0) (unit 1)
+    (in_bom yes) (on_board yes) (dnp no) (fields_autoplaced)
+    (property "Reference" "#PWR038" (at 181.61 91.44 0)
+      (effects (font (size 1.27 1.27)) hide)
+    )
+    (property "Value" "VDD" (at 181.61 82.55 0)
+      (effects (font (size 1.27 1.27)))
+    )
+    (property "Footprint" "" (at 181.61 87.63 0)
+      (effects (font (size 1.27 1.27)) hide)
+    )
+    (property "Datasheet" "" (at 181.61 87.63 0)
+      (effects (font (size 1.27 1.27)) hide)
+    )
+    (pin "1")
+    (instances
+      (project "PD_Micro"
+        (path "/e63e39d7-6ac0-4ffd-8aa3-1841a4541b55"
+          (reference "#PWR038") (unit 1)
+        )
+      )
+    )
+  )
   (symbol (lib_id "-Chip:TPS62175DQC") (at 212.09 49.53 0) (unit 1)
     (in_bom yes) (on_board yes) (dnp no)
@@
     )
   )
+  (symbol (lib_name "R_3") (lib_id "-Passive:R") (at 185.42 83.82 0) (unit 1)
+    (in_bom yes) (on_board yes) (dnp no)
+    (property "Reference" "R16" (at 176.53 81.28 0)
+      (effects (font (size 1.27 1.27)) (justify left))
+    )
+    (property "Value" "10m" (at 176.53 85.09 0)
+      (effects (font (size 1.016 1.016)) (justify left))
+    )
+    (property "Footprint" "Capacitor_SMD:C_1206_3216Metric" (at 186.436 84.074 90)
+      (effects (font (size 1.27 1.27)) hide)
+    )
+    (property "Datasheet" "" (at 185.42 83.82 0)
+      (effects (font (size 1.27 1.27)) hide)
+    )
+    (pin "1")
+    (pin "2")
+    (instances
+      (project "PD_Micro"
+        (path "/e63e39d7-6ac0-4ffd-8aa3-1841a4541b55"
+          (reference "R16") (unit 1)
+        )
+      )
+    )
+  )
   (symbol (lib_id "Switch:SW_DPST_x2") (at 116.84 153.67 0) (unit 1)
     (in_bom yes) (on_board yes) (dnp no)
@@
     )
   )
+  (symbol (lib_id "power:VDD") (at 66.04 64.77 270) (unit 1)
+    (in_bom yes) (on_board yes) (dnp no) (fields_autoplaced)
+    (property "Reference" "#PWR029" (at 62.23 64.77 0)
+      (effects (font (size 1.27 1.27)) hide)
+    )
+    (property "Value" "VDD" (at 69.85 64.77 90)
+      (effects (font (size 1.27 1.27)) (justify left))
+    )
+    (property "Footprint" "" (at 66.04 64.77 0)
+      (effects (font (size 1.27 1.27)) hide)
+    )
+    (property "Datasheet" "" (at 66.04 64.77 0)
+      (effects (font (size 1.27 1.27)) hide)
+    )
+    (pin "1")
+    (instances
+      (project "PD_Micro"
+        (path "/e63e39d7-6ac0-4ffd-8aa3-1841a4541b55"
+          (reference "#PWR029") (unit 1)
+        )
+      )
+    )
+  )
   (symbol (lib_id "-Flag:GND") (at 189.23 104.14 0) (unit 1)
     (in_bom yes) (on_board yes) (dnp no)
@@
     )
   )
-  (symbol (lib_id "power:+3.3V") (at 269.24 41.91 0) (unit 1)
+  (symbol (lib_id "power:+3.3V") (at 257.81 41.91 270) (unit 1)
     (in_bom yes) (on_board yes) (dnp no) (fields_autoplaced)
-    (property "Reference" "#PWR037" (at 269.24 45.72 0)
+    (property "Reference" "#PWR037" (at 254 41.91 0)
       (effects (font (size 1.27 1.27)) hide)
     )
-    (property "Value" "+3.3V" (at 269.24 36.83 0)
-      (effects (font (size 1.27 1.27)))
+    (property "Value" "+3.3V" (at 261.62 41.91 90)
+      (effects (font (size 1.27 1.27)) (justify left))
     )
-    (property "Footprint" "" (at 269.24 41.91 0)
+    (property "Footprint" "" (at 257.81 41.91 0)
       (effects (font (size 1.27 1.27)) hide)
     )
-    (property "Datasheet" "" (at 269.24 41.91 0)
+    (property "Datasheet" "" (at 257.81 41.91 0)
       (effects (font (size 1.27 1.27)) hide)
     )
@@
     )
   )
+  (symbol (lib_id "power:+3.3V") (at 200.66 49.53 90) (unit 1)
+    (in_bom yes) (on_board yes) (dnp no)
+    (property "Reference" "#PWR018" (at 204.47 49.53 0)
+      (effects (font (size 1.27 1.27)) hide)
+    )
+    (property "Value" "+3.3V" (at 200.66 46.99 90)
+      (effects (font (size 1.27 1.27)) (justify left))
+    )
+    (property "Footprint" "" (at 200.66 49.53 0)
+      (effects (font (size 1.27 1.27)) hide)
+    )
+    (property "Datasheet" "" (at 200.66 49.53 0)
+      (effects (font (size 1.27 1.27)) hide)
+    )
+    (pin "1")
+    (instances
+      (project "PD_Micro"
+        (path "/e63e39d7-6ac0-4ffd-8aa3-1841a4541b55"
+          (reference "#PWR018") (unit 1)
+        )
+      )
+    )
+  )
   (symbol (lib_name "C_2") (lib_id "-Passive:C") (at 193.04 55.88 0) (unit 1)
     (in_bom yes) (on_board yes) (dnp no) (fields_autoplaced)
@@
     )
   )
-  (symbol (lib_id "-Flag:+5V") (at 200.66 49.53 90) (unit 1)
-    (in_bom yes) (on_board yes) (dnp no)
-    (property "Reference" "#PWR018" (at 204.47 49.53 0)
-      (effects (font (size 1.27 1.27)) hide)
+  (symbol (lib_name "R_1") (lib_id "-Passive:R") (at 99.06 128.27 90) (unit 1)
+    (in_bom yes) (on_board yes) (dnp no) (fields_autoplaced)
+    (property "Reference" "R11" (at 99.06 121.92 90)
+      (effects (font (size 1.27 1.27)))
     )
-    (property "Value" "+5V" (at 198.12 49.53 90)
-      (effects (font (size 1.27 1.27)) (justify left))
+    (property "Value" "5.1k" (at 99.06 124.46 90)
+      (effects (font (size 1.016 1.016)))
     )
-    (property "Footprint" "" (at 200.66 49.53 0)
+    (property "Footprint" "Resistor_SMD:R_0805_2012Metric" (at 99.314 127.254 90)
       (effects (font (size 1.27 1.27)) hide)
     )
-    (property "Datasheet" "" (at 200.66 49.53 0)
+    (property "Datasheet" "" (at 99.06 128.27 0)
       (effects (font (size 1.27 1.27)) hide)
     )
     (pin "1")
+    (pin "2")
     (instances
       (project "PD_Micro"
         (path "/e63e39d7-6ac0-4ffd-8aa3-1841a4541b55"
-          (reference "#PWR018") (unit 1)
+          (reference "R11") (unit 1)
         )
       )
     )
   )
-  (symbol (lib_name "R_1") (lib_id "-Passive:R") (at 99.06 128.27 90) (unit 1)
+  (symbol (lib_id "power:VDD") (at 64.77 87.63 270) (unit 1)
     (in_bom yes) (on_board yes) (dnp no) (fields_autoplaced)
-    (property "Reference" "R11" (at 99.06 121.92 90)
-      (effects (font (size 1.27 1.27)))
+    (property "Reference" "#PWR030" (at 60.96 87.63 0)
+      (effects (font (size 1.27 1.27)) hide)
     )
-    (property "Value" "5.1k" (at 99.06 124.46 90)
-      (effects (font (size 1.016 1.016)))
+    (property "Value" "VDD" (at 68.58 87.63 90)
+      (effects (font (size 1.27 1.27)) (justify left))
     )
-    (property "Footprint" "Resistor_SMD:R_0805_2012Metric" (at 99.314 127.254 90)
+    (property "Footprint" "" (at 64.77 87.63 0)
       (effects (font (size 1.27 1.27)) hide)
     )
-    (property "Datasheet" "" (at 99.06 128.27 0)
+    (property "Datasheet" "" (at 64.77 87.63 0)
       (effects (font (size 1.27 1.27)) hide)
     )
     (pin "1")
-    (pin "2")
     (instances
       (project "PD_Micro"
         (path "/e63e39d7-6ac0-4ffd-8aa3-1841a4541b55"
-          (reference "R11") (unit 1)
+          (reference "#PWR030") (unit 1)
         )
       )
@@
       (effects (font (size 1.27 1.27)) (justify left))
     )
-    (property "Footprint" "-Connector:TerminalBlock_3.5mm_2P" (at 30.48 22.86 0)
+    (property "Footprint" "TerminalBlock:TerminalBlock_bornier-2_P5.08mm" (at 30.48 22.86 0)
       (effects (font (size 1.27 1.27)) hide)
     )

Commit message: a few fixes
Parts:
- J2, J3, J4, J5: footprint Connector_PinHeader_1.00mm:PinHeader_1x02_P1.00mm_Vertical -> Connector_PinHeader_2.54mm:PinHeader_1x02_P2.54mm_Vertical
Changed lines of the file:
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@@
       (effects (font (size 1.27 1.27)) (justify left))
     )
-    (property "Footprint" "Connector_PinHeader_1.00mm:PinHeader_1x02_P1.00mm_Vertical" (at 144.78 69.85 0)
+    (property "Footprint" "Connector_PinHeader_2.54mm:PinHeader_1x02_P2.54mm_Vertical" (at 144.78 69.85 0)
       (effects (font (size 1.27 1.27)) hide)
     )
@@
       (effects (font (size 1.27 1.27)) (justify left))
     )
-    (property "Footprint" "Connector_PinHeader_1.00mm:PinHeader_1x02_P1.00mm_Vertical" (at 144.78 82.55 0)
+    (property "Footprint" "Connector_PinHeader_2.54mm:PinHeader_1x02_P2.54mm_Vertical" (at 144.78 82.55 0)
       (effects (font (size 1.27 1.27)) hide)
     )
@@
       (effects (font (size 1.27 1.27)) (justify left))
     )
-    (property "Footprint" "Connector_PinHeader_1.00mm:PinHeader_1x02_P1.00mm_Vertical" (at 144.78 76.2 0)
+    (property "Footprint" "Connector_PinHeader_2.54mm:PinHeader_1x02_P2.54mm_Vertical" (at 144.78 76.2 0)
       (effects (font (size 1.27 1.27)) hide)
     )
@@
       (effects (font (size 1.27 1.27)) (justify left))
     )
-    (property "Footprint" "Connector_PinHeader_1.00mm:PinHeader_1x02_P1.00mm_Vertical" (at 144.78 63.5 0)
-      (effects (font (size 1.27 1.27)) hide)
-    )
+    (property "Footprint" "Connector_PinHeader_2.54mm:PinHeader_1x02_P2.54mm_Vertical" (at 144.78 63.5 0)
+      (effects (font (size 1.27 1.27)) hide)
+    )
