File: PD_Micro.kicad_sch (KiCad schematic)
At the start: 52 parts, among them J1 Conn_01x02, J2 Conn_01x02, J3 USB_C_Receptacle_USB2.0, J4 Conn_01x02, J5 Conn_01x02, J7 Conn_01x02, J8 Conn_01x02, Q2 DTC143E, Q4 IRF9393, SW1 SW_DIP_x06, SW2 SW_DPST_x2, SW3 SW_Push, SW4 SW_Push, SW5 SW_DPST_x2, U1 SRV05-4, U2 Pico, U3 TMCS1108, U6 oledSym, U7 LMR54410

Commit message: v3.1 finished
Parts:
- removed C8: 10uF, Capacitor_SMD:C_0805_2012Metric, symbol -Passive:C
- removed Q2: DTC143E, -Discrete:SOT-323_SC-70, symbol -Discrete:DTC143E
- added C11: 1uF 50V, Capacitor_SMD:C_0805_2012Metric, symbol -Passive:C
- added Q1: BC847, Package_TO_SOT_SMD:SOT-23, symbol PCM_Transistor_BJT_AKL:BC847
- added R12: 20m, Capacitor_SMD:C_1206_3216Metric, symbol -Passive:R
- added R5, R7: 4k7, Resistor_SMD:R_0805_2012Metric, symbol -Passive:R
- C10: value 22u -> 22u 50V
- C12: value 10u -> 10u 50V
- C3: value 2.2u -> 2.2u 50V
- Q4: footprint Package_SO_AKL:SO-8_3.9x4.9mm_P1.27mm -> Package_SO:SOIC-8_3.9x4.9mm_P1.27mm
- R16: value 10m -> 20m
- U3: footprint PCM_4ms_Package_SOIC:SOIC-8_3.9x4.9mm_Pitch1.27mm -> Package_SO:SOIC-8_3.9x4.9mm_P1.27mm
- U6: footprint OLED094:SSD1306_0.96_Oled -> SSD1306:128x64OLED
Connections:
- net +5V: now also C11.1
- net ENOUT: now also R7.1
- net GND: now also U3.6 (NC), C11.2, Q1.2 (E), R5.1
- net VBUS: now also R12.1
- net VDD: now also R12.2
- net at R8.2: now also Q1.3 (C)
- net SW: now reaches C5.2, L1.1, U7.6 (SW)
- new net: Q1.1 (B), R5.2, R7.2
- no-connect marks 4 -> 3

Commit message: finished
Parts:
- added J6: Conn_01x07, Connector_PinSocket_2.54mm:PinSocket_1x07_P2.54mm_Vertical, symbol Connector_Generic:Conn_01x07
Connections:
- net EN12V: now also J6.5 (Pin_5)
- net EN15V: now also J6.4 (Pin_4)
- net EN20V: now also J6.3 (Pin_3)
- net EN5V: now also J6.7 (Pin_7)
- net EN9V: now also J6.6 (Pin_6)
- net ENOUT: now also J6.2 (Pin_2)
- net GND: now also J6.1 (Pin_1)
Other:
- moved on the sheet: D2

Commit message: final
Parts:
- U4: value ~ -> AP33772
Connections:
- net SW_OUT: now reaches SW2.2 (B), U2.16 (GPIO12)
- net SW_VA: now reaches SW5.2 (B), U2.17 (GPIO13)
- net BTN_DOWN: now reaches SW4.2, U2.19 (GPIO14)
- net BTN_UP: now reaches SW3.2, U2.20 (GPIO15)
- net LED: now reaches D2.4 (DIN), U2.5 (GPIO3)
Other:
- note added: "5V Regulator"
- note added: "Buttons"
- note added: "ESD Protection"
- note added: "External Triggers"
- note added: "Hallsensor"
- note added: "LED"
- note added: "Mountingholes"
- note added: "Output"
- note added: "Output Mosfet"
- note added: "Pins"
- note added: "PoverDelivery IC"
- note added: "Pullups/down"
- note added: "Switches"
- note added: "USB-C"
- note removed: "5V 9V 12V 15V 20V Power Supply Mode"
- note removed: "USB-C socket"
- company: (none) -> HTL Rankweil
- title: (none) -> USBC_PD-Trigger
- moved on the sheet: C1, C10, C11, C12, C13, C14, C15, C2, C3, C4, C5, C6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
