File: PD_Micro-rounded.kicad_pcb (KiCad board)
At the start: 2 copper layers, 62 x 53 mm, 43 parts, among them J1 Conn_01x02, Q1 DMP3017SFK, Q2 DTC143E, SW1 SW_DIP_x06, SW2 SW_DPST_x2, SW3 SW_Push, SW4 SW_Push, SW5 SW_DPST_x2, U1 SRV05-4, U2 Pico, U3 TPS62175DQC, U4 FUSB302BMPX, U5 ACS723xMATR-10AB, U6 oledSym

Commit message: pcb
Routing:
- net SCL: track 27.3 -> 26.4 mm
- net /D1_P: track 18.9 -> 18.2 mm
- net ADC0: track 40.8 -> 40.2 mm
- net SDA: track 20.9 -> 20.3 mm
