File: PD_Micro-Schul-Laptop.kicad_sch (KiCad schematic)
At the start: 48 parts, among them J1 Conn_01x02, J2 Conn_01x02, J4 Conn_01x02, J5 Conn_01x02, Q1 DMP3017SFK, Q2 DTC143E, SW1 SW_DIP_x06, SW2 SW_DPST_x2, SW3 SW_Push, SW4 SW_Push, SW5 SW_DPST_x2, U1 SRV05-4, U2 Pico, U5 ACS723xLCTR-10AB, U6 oledSym, U7 NE5532

Commit message: usbc-save
Parts:
- removed C13, C15: 100nF, Capacitor_SMD:C_0805_2012Metric, symbol -Passive:C
- removed C14: 1uF, Capacitor_SMD:C_0805_2012Metric, symbol -Passive:C
- removed J2, J4, J5: Conn_01x02, Connector_PinHeader_2.54mm:PinHeader_1x02_P2.54mm_Vertical, symbol -Connector:Conn_01x02
- removed R10, R11: 5.1k, Resistor_SMD:R_0805_2012Metric, symbol -Passive:R
- removed R16: 10m, Capacitor_SMD:C_1206_3216Metric, symbol -Passive:R
- removed TH1: NTC-10k, Resistor_SMD:R_0805_2012Metric, symbol Device:Thermistor
- removed TP1, TP2, TP3, TP4: TestPoint, Connector_PinHeader_2.54mm:PinHeader_1x01_P2.54mm_Vertical, symbol -Connector:TestPoint
- removed U4: ~, Package_DFN_QFN:WQFN-24-1EP_4x4mm_P0.5mm_EP2.6x2.6mm_ThermalVias, symbol AP33772:AP33772
- removed U7: NE5532, PCM_4ms_Package_SOIC:SOIC-8-1EP_3.9x4.9mm_Pitch1.27mm, symbol Amplifier_Operational:NE5532
- added C10: 0.1uF, Capacitor_SMD:C_0805_2012Metric, symbol -Passive:C
- added C11, C9: 10uF, Capacitor_SMD:C_0805_2012Metric, symbol -Passive:C
- added C5: 330pF, Capacitor_SMD:C_0805_2012Metric, symbol -Passive:C
- added L1: 10uH, -Passive:L_4012, symbol -Passive:L_cored
- added R2, R3: 22R, Resistor_SMD:R_0805_2012Metric, symbol -Passive:R
- added R5: 51k, Resistor_SMD:R_0805_2012Metric, symbol -Passive:R
- added R7: 270k, Resistor_SMD:R_0805_2012Metric, symbol -Passive:R
- added U3: TPS62175DQC, -Chip:WSON-10-1EP_2x3mm_P0.5mm_EP0.84x2.4mm, symbol -Chip:TPS62175DQC
- added U4: FUSB302BMPX, -Chip:WQFN-14-1EP_2.5x2.5mm_P0.5mm_EP1.45x1.45mm, symbol -Chip:FUSB302BMPX
- C12: value 10u -> 0.1uF
- C3: value 1uF -> 330pF
- J1: footprint TerminalBlock:TerminalBlock_bornier-2_P5.08mm -> -Connector:TerminalBlock_3.5mm_2P
- R4, R9: value 5.1k -> 2k
- USB1: footprint USB-C:HRO-TYPE-C-31-M-12 -> -Connector:HRO-TYPE-C-31-M-12
Connections:
- net +5V: now also C12.1, C11.1, C9.1, L1.2, R7.1, U3.10 (VOS), U3.8 (~{SLEEP}), U4.12 (VCONN), U4.13 (VCONN), U4.3 (VDD), U4.4 (VDD)
- net CC1: now also U1.3 (IO2), C5.2, U4.1 (CC2), U4.14 (CC2); no longer U1.1 (IO1)
- net CC2: now also C3.2, U1.1 (IO1), U4.10 (CC1), U4.11 (CC1); no longer U1.3 (IO2)
- net D_N: now also R3.2; no longer U1.6 (IO4), U2.42 (USB_DM)
- net D_P: now also R2.2; no longer U1.4 (IO3), U2.41 (USB_DP)
- net GND: now also C3.1, C10.2, C11.2, C5.1, C9.2, R5.2, U3.1 (PGND), U3.11 (PAD), U3.4 (NC), U3.6 (AGND), U4.15 (GND), U4.8 (GND), U4.9 (GND); no longer C3.2
- net SCL: now also U2.10 (GPIO7), U4.6 (SCL); no longer U2.7 (GPIO5)
- net SDA: now also U2.9 (GPIO6), U4.7 (SDA); no longer U2.6 (GPIO4)
- net VBUS: now also USB1.11 (VBUS), USB1.2 (VBUS), C10.1, U3.2 (VIN), U3.3 (EN), U4.2 (VBUS)
- net at SW2.2 (B): now also U2.6 (GPIO4); no longer U2.9 (GPIO6)
- removed net VDD: C12.1, C3.1, USB1.11 (VBUS), USB1.2 (VBUS)
- new net: R5.1, R7.2, U3.5 (FB)
- new net D1_N: R3.1, U1.6 (IO4), U2.42 (USB_DM)
- new net D1_P: R2.1, U1.4 (IO3), U2.41 (USB_DP)
- new net INT_N: U2.7 (GPIO5), U4.5 (INT_N)
- new net SW1: L1.1, U3.9 (SW)
Other:
- note added: "4.5-28V to 5V DC-DC"
- note added: "I2C Address: 0x22"
- note removed: "DIP Switches"
- moved on the sheet: C8, SW1
