File: PD_Micro.kicad_pcb (KiCad board)
At the start: 2 copper layers, 62 x 53 mm, 46 parts, among them J1 Conn_01x02, Q1 DMP3017SFK, Q2 DTC143E, SW1 SW_DIP_x06, SW2 SW_DPST_x2, SW3 SW_Push, SW4 SW_Push, SW5 SW_DPST_x2, U1 SRV05-4, U2 Pico, U3 TPS62175DQC, U4 FUSB302BMPX, U5 ACS723xLCTR-10AB, U6 oledSym

Commit message: bevore rebuild
Parts:
- removed the G*** at (188.6, 125.9)
- removed the G*** at (206.9, 118.2)
Other:
- board text added: "HTL-Rankweil 4AHEL Manuel Mayrhofer Johannes Melcher-Millner USBC_PD-Trigger v1.0"
- board text removed: "HTL-Rankweil 4AHEL Manuel Mayrhofer Johannes Melcher-Millner USBC_PD-Trigger"

Commit message: sch finished, parts placed
Parts:
- removed C12: 0.1uF, Capacitor_SMD:C_0805_2012Metric
- removed C5: 330pF, Capacitor_SMD:C_0805_2012Metric
- added C13: 100nF, Capacitor_SMD:C_0805_2012Metric, F.Cu at (192.7, 105.0)
- added C14: 1uF, Capacitor_SMD:C_0805_2012Metric, F.Cu at (195.0, 99.4)
- added C15: 100nF, Capacitor_SMD:C_0805_2012Metric, F.Cu at (195.0, 103.1)
- added C16: 2.2u, Capacitor_SMD:C_0805_2012Metric, F.Cu at (223.7, 104.2)
- added J2: Conn_01x02, Connector_PinHeader_1.00mm:PinHeader_1x02_P1.00mm_Vertical, F.Cu at (227.5, 117.8)
- added J3: Conn_01x02, Connector_PinHeader_1.00mm:PinHeader_1x02_P1.00mm_Vertical, F.Cu at (232.6, 117.8)
- added J4: Conn_01x02, Connector_PinHeader_1.00mm:PinHeader_1x02_P1.00mm_Vertical, F.Cu at (230.0, 117.8)
- added J5: Conn_01x02, Connector_PinHeader_1.00mm:PinHeader_1x02_P1.00mm_Vertical, F.Cu at (235.1, 117.8)
- added L2: 10uH, -Passive:L_4012, F.Cu at (223.8, 96.2)
- added R10: 5.1k, Resistor_SMD:R_0805_2012Metric, F.Cu at (185.7, 101.0)
- added R11: 5.1k, Resistor_SMD:R_0805_2012Metric, F.Cu at (185.7, 99.0)
- added R12: 270k, Resistor_SMD:R_0805_2012Metric, F.Cu at (219.3, 106.0)
- added R13: 100k, Resistor_SMD:R_0805_2012Metric, F.Cu at (224.0, 106.9)
- added R14: 30k, Resistor_SMD:R_0805_2012Metric, F.Cu at (219.3, 103.6)
- added TH1: Thermistor, Resistor_SMD:R_0805_2012Metric, F.Cu at (185.7, 103.0)
- added TP1: TestPoint, Connector_PinHeader_1.00mm:PinHeader_1x01_P1.00mm_Vertical, F.Cu at (229.9, 114.0)
- added TP2: TestPoint, Connector_PinHeader_1.00mm:PinHeader_1x01_P1.00mm_Vertical, F.Cu at (232.4, 114.0)
- added TP3: TestPoint, TestPoint:TestPoint_Pad_D1.0mm, F.Cu at (222.8, 114.1)
- added U7: ~, Package_DFN_QFN:WQFN-24-1EP_4x4mm_P0.5mm_EP2.6x2.6mm, F.Cu at (190.6, 100.2)
- C3: value 330pF -> 22u
- R4, R9: value 2k -> 5.1k
- U4: value FUSB302BMPX -> TPS62175DQC; footprint -Chip:WQFN-14-1EP_2.5x2.5mm_P0.5mm_EP1.45x1.45mm -> -Chip:WSON-10-1EP_2x3mm_P0.5mm_EP0.84x2.4mm
- moved C3 30.3 mm to (215.5, 103.6)
- moved U4 29.6 mm to (223.7, 101.3)
- moved U1 5.07 mm to (188.3, 106.2), turned to 0 degrees
- moved G*** 1.93 mm to (234.2, 108.8)
- moved R1 0.25 mm to (183.6, 105.1)
Connections:
- C3 pad 1: GND -> +3.3V
- C3 pad 2: /CC2 -> GND
- R4 pad 1: +5V -> +3.3V
- R9 pad 1: +5V -> +3.3V
- U1 pad 1: /CC2 -> CC2
- U1 pad 3: /CC1 -> CC1
- U4 pad 1: /CC1 -> GND
- U4 pad 10: /CC2 -> +3.3V
- U4 pad 11: /CC2 -> GND
- U4 pad 3: +5V -> VBUS
- U4 pad 4: +5V -> GND
- U4 pad 5: INT_N -> Net-(U4-FB)
- U4 pad 6: SCL -> GND
- U4 pad 7: SDA -> Net-(U4-PG)
- U4 pad 8: GND -> +5V
- U4 pad 9: GND -> /SW1
- USB1 pad 10: /CC2 -> CC2
- USB1 pad 4: /CC1 -> CC1
Routing:
- net /CC1: track 14.5 -> 0.00 mm, vias 3 -> 0
- net /CC2: track 14.5 -> 0.00 mm, vias 3 -> 0
- net /D1_P: track 18.9 -> 5.72 mm
- net /D1_N: track 18.8 -> 5.76 mm
- net SDA: track 20.9 -> 8.81 mm, vias 1 -> 0
- net SCL: track 27.7 -> 15.9 mm, vias 1 -> 0
- net INT_N: track 10.2 -> 0.00 mm, vias 1 -> 0
- net GND: track 18.9 -> 8.71 mm, vias 8 -> 6
- net +5V: track 12.1 -> 5.46 mm, vias 8 -> 6
- net VBUS: track 13.0 -> 6.99 mm, vias 15 -> 12
- net +3.3V: track 0.00 -> 4.80 mm
- net Net-(U7-V3VD): track 0.00 -> 3.85 mm
- net EN9V: track 12.2 -> 11.5 mm
- net unconnected-(U2-GPIO1-Pad2): track 0.51 -> 0.00 mm
Other:
- board text added: "CC1"
- board text added: "CC2"
- board text added: "OUTEN"
- board text added: "VBUS 5V 3.3V GND"

Commit message: pcb v2 finished
Parts:
- R12: value 270k -> 30k
- R14: value 30k -> 10k
- moved TP3 248.9 mm to (1.02, 1.02)
- moved TH1 7.97 mm to (193.4, 104.8), turned to -90 degrees
- moved L2 4.39 mm to (226.2, 99.9), turned to 90 degrees
- moved D1 4.32 mm to (211.6, 102.0)
- moved C15 4.06 mm to (191.3, 104.8), turned to -90 degrees
- moved C13 3.80 mm to (195.8, 102.9)
- moved TP2 3.05 mm to (229.4, 114.0)
- moved U5 2.44 mm to (215.9, 97.0)
- moved C3 2.41 mm to (215.5, 106.0)
- moved TP1 2.03 mm to (231.9, 114.0)
- moved U4 1.62 mm to (222.5, 102.4)
- moved C16 1.09 mm to (223.3, 105.2), turned to 180 degrees
- moved R13 0.92 mm to (223.3, 107.4)
- moved C1 0.89 mm to (183.7, 107.1)
- moved R14 0.18 mm to (219.2, 103.4), turned to 180 degrees
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Connections:
- L1 pad 1: /SW1 -> Net-(U3-SW)
- L2 pad 1: /SW1 -> Net-(U4-SW)
- U2 pad 20: Net-(U2-GPIO15) -> unconnected-(U2-GPIO15-Pad20)
- U3 pad 9: /SW1 -> Net-(U3-SW)
- U4 pad 9: /SW1 -> Net-(U4-SW)
Routing:
- net CC2: track 0.00 -> 75.8 mm, vias 0 -> 3
- net CC1: track 0.00 -> 75.2 mm, vias 0 -> 4
- net +3.3V: track 4.80 -> 71.4 mm
- net VBUS: track 6.99 -> 69.5 mm, vias 12 -> 14
- net GND: track 8.71 -> 33.5 mm, vias 6 -> 15
- net SDA: track 8.81 -> 26.8 mm, vias 0 -> 1
- net SCL: track 15.9 -> 33.8 mm, vias 0 -> 1
- net /D1_N: track 5.76 -> 22.5 mm
- net Net-(U4-PG): track 0.00 -> 9.90 mm
- net /D1_P: track 5.72 -> 14.3 mm
- net Net-(U3-SW): track 0.00 -> 5.39 mm, vias 0 -> 2
- net /SW1: track 5.39 -> 0.00 mm, vias 2 -> 0
- net +5V: track 5.46 -> 10.2 mm, vias 6 -> 15
- net Net-(U7-VSV): track 0.00 -> 4.53 mm
- net Net-(U4-FB): track 0.00 -> 4.03 mm
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- added copper zone on B.Cu, net /SHIELD

Commit message: v2.1
Parts:
- removed TP3: TestPoint, TestPoint:TestPoint_Pad_D1.0mm
- added C5: 2.2u, Capacitor_SMD:C_0805_2012Metric, F.Cu at (215.4, 104.7)
- added R15: 100k, Resistor_SMD:R_0805_2012Metric, F.Cu at (203.8, 98.2)
- R12: value 30k -> 270k
- R14: value 10k -> 30k
- U7: footprint Package_DFN_QFN:WQFN-24-1EP_4x4mm_P0.5mm_EP2.6x2.6mm -> Package_DFN_QFN:WQFN-24-1EP_4x4mm_P0.5mm_EP2.6x2.6mm_ThermalVias
- moved C8 10.3 mm to (211.8, 105.3)
- moved C11 10.3 mm to (211.8, 107.4)
- moved L1 3.81 mm to (203.8, 101.7), turned to 0 degrees
- moved C9 2.07 mm to (204.4, 105.2), turned to 180 degrees
- moved R14 1.30 mm to (219.0, 104.7)
- moved R12 0.96 mm to (219.0, 106.9)
- moved C3 0.89 mm to (215.4, 106.9)
- moved Q2 0.85 mm to (207.5, 100.6)
Connections:
- U3 pad 7: unconnected-(U3-PG-Pad7) -> Net-(U3-PG)
Routing:
- net +5V: track 10.2 -> 15.5 mm, vias 15 -> 16
- net Net-(U3-SW): track 5.39 -> 8.50 mm
- net Net-(U3-PG): track 0.00 -> 2.83 mm
- net GND: track 33.5 -> 35.4 mm, vias 15 -> 16
- net VBUS: track 69.5 -> 70.7 mm, vias 14 -> 15
- net +3.3V: track 71.4 -> 70.4 mm
- net Net-(Q2-C): track 2.28 -> 1.67 mm
Other:
- board text added: "HTL-Rankweil 4AHEL Manuel Mayrhofer Johannes Melcher-Millner USBC_PD-Trigger v2.1"
- board text removed: "HTL-Rankweil 4AHEL Manuel Mayrhofer Johannes Melcher-Millner USBC_PD-Trigger v1.0"

Commit message: v2.2
Parts:
- added R16: 10m, Capacitor_SMD:C_1206_3216Metric, F.Cu at (180.5, 95.2)
- J1: footprint -Connector:TerminalBlock_3.5mm_2P -> TerminalBlock:TerminalBlock_bornier-2_P5.08mm
- moved G*** 18.6 mm to (230.6, 90.5)
- moved J1 2.19 mm to (232.6, 98.9)
- moved R11 0.64 mm to (185.6, 99.6)
- moved R10 0.64 mm to (185.6, 101.7)
Connections:
- U4 pad 8: +5V -> +3.3V
- U7 pad 1: VBUS -> VDD
- USB1 pad 11: VBUS -> VDD
- USB1 pad 2: VBUS -> VDD
Routing:
- net VDD: track 0.00 -> 21.9 mm, vias 0 -> 2
- net +3.3V: track 70.4 -> 75.2 mm, vias 0 -> 1
- net +5V: track 15.5 -> 10.7 mm, vias 16 -> 14
- net VBUS: track 70.7 -> 66.7 mm, vias 15 -> 13
- net CC1: track 75.2 -> 74.2 mm
- net GND: vias 16 -> 15
Other:
- board text added: "GND"
- board text added: "Vout"

Commit message: a few fixes
Parts:
- J2, J3, J4, J5: footprint Connector_PinHeader_1.00mm:PinHeader_1x02_P1.00mm_Vertical -> Connector_PinHeader_2.54mm:PinHeader_1x02_P2.54mm_Vertical
- moved J5 8.02 mm to (228.1, 113.8), turned to 90 degrees
- moved TP1 3.30 mm to (231.9, 110.7)
- moved TP2 3.30 mm to (229.4, 110.7)
- moved J3 1.28 mm to (233.8, 117.7)
- moved J2 1.15 mm to (226.3, 117.7)
- moved J4 0.13 mm to (230.0, 117.7)
Routing:
- net CC2: track 75.6 -> 68.0 mm
- net CC1: track 74.2 -> 70.8 mm
- net +3.3V: track 75.2 -> 72.4 mm
- net VBUS: track 66.7 -> 69.3 mm
- net Net-(Q1-G): track 21.1 -> 22.3 mm
- net /OUT: vias 16 -> 8
- net +5V: vias 14 -> 11

Commit message: v3
Parts:
- removed C10: 0.1uF, Capacitor_SMD:C_0805_2012Metric
- removed C11, C9: 10uF, Capacitor_SMD:C_0805_2012Metric
- removed C16, C5: 2.2u, Capacitor_SMD:C_0805_2012Metric
- removed G***: LOGO, LOGO
- removed J3: Conn_01x02, Connector_PinHeader_2.54mm:PinHeader_1x02_P2.54mm_Vertical
- removed L1, L2: 10uH, -Passive:L_4012
- removed R12, R7: 270k, Resistor_SMD:R_0805_2012Metric
- removed R13, R15: 100k, Resistor_SMD:R_0805_2012Metric
- removed R14: 30k, Resistor_SMD:R_0805_2012Metric
- removed R2, R3: 22R, Resistor_SMD:R_0805_2012Metric
- removed R5: 51k, Resistor_SMD:R_0805_2012Metric
- removed U3: TPS62175DQC, -Chip:WSON-10-1EP_2x3mm_P0.5mm_EP0.84x2.4mm
- removed the U4 at (222.5, 102.4)
- added C12: 10u, Capacitor_SMD:C_0805_2012Metric, F.Cu at (184.3, 95.7)
- added TP3: TestPoint, Connector_PinHeader_2.54mm:PinHeader_1x01_P2.54mm_Vertical, F.Cu at (233.4, 121.4)
- added TP4: TestPoint, Connector_PinHeader_2.54mm:PinHeader_1x01_P2.54mm_Vertical, F.Cu at (233.4, 117.6)
- added U7: NE5532, PCM_4ms_Package_SOIC:SOIC-8-1EP_3.9x4.9mm_Pitch1.27mm, F.Cu at (200.9, 99.7)
- C3: value 22u -> 1uF
- TH1: value Thermistor -> NTC-10k
- TP1, TP2: footprint Connector_PinHeader_1.00mm:PinHeader_1x01_P1.00mm_Vertical -> Connector_PinHeader_2.54mm:PinHeader_1x01_P2.54mm_Vertical
- moved C4 27.8 mm to (212.4, 98.0), turned to -90 degrees
- moved J2 25.4 mm to (230.7, 92.6), turned to 90 degrees
- moved C6 23.8 mm to (210.4, 98.0), turned to -90 degrees
- moved R6 21.2 mm to (214.5, 98.0), turned to -90 degrees
- moved C2 19.7 mm to (208.4, 98.0), turned to -90 degrees
- moved C3 12.7 mm to (206.3, 98.0), turned to -90 degrees
- moved TP1 11.8 mm to (227.0, 121.4), turned to 90 degrees
- moved C14 11.8 mm to (205.7, 104.3)
- moved R16 11.1 mm to (191.5, 96.2)
- moved C7 10.6 mm to (220.5, 98.0), turned to 0 degrees
- moved Q1 7.57 mm to (217.1, 97.6)
- moved C15 7.36 mm to (198.6, 104.1), turned to 0 degrees
- moved TP2 7.32 mm to (227.0, 117.6), turned to 90 degrees
- moved R8 7.22 mm to (213.0, 101.5)
- moved C8 6.27 mm to (207.4, 100.9)
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- renumbered U7 to U4
Connections:
- C13 pad 1: Net-(U7-IFB) -> Net-(U4-V3VD)
- C15 pad 1: Net-(U7-V3VD) -> Net-(U4-IFB)
- C3 pad 1: +3.3V -> VDD
- D1 pad 1: /OUT -> OUT
- J1 pad 1: /OUT -> OUT
- J2 pad 1: VBUS -> OUT
- J2 pad 2: VBUS -> OUT
- R4 pad 1: +3.3V -> +5V
- R9 pad 1: +3.3V -> +5V
- TP1 pad 1: CC1 -> CC2
- TP2 pad 1: CC2 -> CC1
- U1 pad 1: CC2 -> CC1
- U1 pad 3: CC1 -> CC2
- U1 pad 4: /D1_P -> /D_P
- U1 pad 6: /D1_N -> /D_N
- U2 pad 10: SCL -> unconnected-(U2-GPIO7-Pad10)
- U2 pad 41: /D1_P -> /D_P
- U2 pad 42: /D1_N -> /D_N
- U2 pad 6: Net-(SW2A-B) -> SDA
- U2 pad 7: INT_N -> SCL
- U2 pad 9: SDA -> Net-(SW2A-B)
- U4 pad 10: (no net) -> unconnected-(U4-NC-Pad10)
- U4 pad 12: Net-(U7-V3VD) -> Net-(U4-V3VD)
- U4 pad 15: Net-(U7-IFB) -> Net-(U4-IFB)
- U4 pad 18: (no net) -> unconnected-(U4-NC-Pad18)
- U4 pad 19: (no net) -> unconnected-(U4-NC-Pad19)
- U4 pad 2: (no net) -> unconnected-(U4-NC-Pad2)
- U4 pad 21: (no net) -> unconnected-(U4-NC-Pad21)
- U4 pad 22: VBUS -> OUT
- U4 pad 4: SDA -> SCL
- U4 pad 5: SCL -> SDA
- U5 pad 3: /OUT -> OUT
- U5 pad 4: /OUT -> OUT
Routing:
- net +3.3V: track 72.4 -> 0.00 mm, vias 1 -> 0
- net VBUS: track 69.3 -> 4.82 mm, vias 13 -> 9
- net SDA: track 26.8 -> 68.9 mm
- net ENOUT: track 13.1 -> 46.0 mm
- net SCL: track 33.8 -> 65.4 mm, vias 1 -> 2
- net GND: track 35.4 -> 6.68 mm, vias 15 -> 14
- net OUT: track 0.00 -> 23.1 mm, vias 0 -> 15
- net /D1_N: track 22.5 -> 0.00 mm
- net VDD: track 21.9 -> 41.1 mm, vias 2 -> 10
- net Net-(Q1-G): track 22.3 -> 4.51 mm, vias 2 -> 0
- net /D1_P: track 14.3 -> 0.00 mm
- net Net-(U4-V5V): track 4.53 -> 17.1 mm, vias 0 -> 2
- net Net-(U4-PG): track 9.90 -> 0.00 mm
- net Net-(U3-SW): track 8.50 -> 0.00 mm, vias 2 -> 0
- net +5V: track 10.7 -> 18.0 mm, vias 11 -> 6
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- added copper zone on B.Cu, net OUT
- added copper zone on F.Cu, net OUT
- added copper zone on B.Cu, net VDD
- added copper zone on F.Cu, net VDD
- removed copper zone on F.Cu, net +5V
- removed copper zone on B.Cu, net /OUT
- removed copper zone on F.Cu, net /OUT
Other:
- board text added: "HTL-Rankweil 4AHEL Manuel Mayrhofer Johannes Melcher-Millner USBC_PD-Trigger v3.0"
- board text removed: "HTL-Rankweil 4AHEL Manuel Mayrhofer Johannes Melcher-Millner USBC_PD-Trigger v2.1"

Commit message: usbc-save
Parts:
- moved C14 0.41 mm to (206.1, 104.3)
Routing:
- net VDD: track 41.1 -> 40.7 mm, vias 10 -> 8
- net VBUS: vias 9 -> 12
