File: PD-LabSupply.kicad_pcb (KiCad board)
At the start: 2 copper layers, 62 x 53 mm, 56 parts, among them J1 Conn_01x02, J2 Conn_01x02, J3 USB_C_Receptacle_USB2.0, J4 Conn_01x02, J5 Conn_01x02, J6 Conn_01x07, J7 Conn_01x02, J8 Conn_01x02, Q1 BC847, Q4 IRF9393, SW1 SW_DIP_x06, SW2 SW_DPST_x2, SW3 SW_Push, SW4 SW_Push, SW5 SW_DPST_x2, U1 SRV05-4, U2 Pico, U3 TMCS1108, U6 oledSym, U7 LMR54410

Commit message: rename
Other:
- board text added: "PD-LabSupply"
- board text removed: "USBC_PD_Trigger"
Changed lines of the file:
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@@
     (effects (font (size 1 1) (thickness 0.15)))
   )
-  (gr_text "USBC_PD_Trigger" (at 96.5954 36.88) (layer "F.SilkS" knockout)
+  (gr_text "PD-LabSupply" (at 99.2 36.88) (layer "F.SilkS" knockout)
     (effects (font (size 2 2) (thickness 0.3)) (justify left bottom))
   )

Commit message: fine
Parts:
- H1, H2, H3, H4: footprint -Hole:D1_8_PAD -> MountingHole:MountingHole_2.5mm
- U2: footprint MCU_RaspberryPi_and_Boards:RPi_Pico_SMD_TH -> MCU_RaspberryPi_and_Boards:RPi_Pico_THT
- U4: value ~ -> AP33772
- U6: footprint SSD1306:128x64OLED -> SSD1306:SSD1306_0.96_Oled
- moved U6 18.9 mm to (83.8, 85.4)
- moved H3 5.11 mm to (83.0, 80.0)
- moved H1 1.33 mm to (83.0, 35.0)
- moved H2 1.29 mm to (139.4, 35.0)
- moved H4 0.88 mm to (139.3, 84.8)
- moved SW4 0.87 mm to (136.1, 79.2)
- moved J5 0.77 mm to (135.4, 57.9)
- moved J2 0.76 mm to (135.4, 39.6)
- moved SW2 0.54 mm to (115.8, 85.4)
- moved SW5 0.52 mm to (125.9, 85.4)
Routing:
- net CC1: track 70.4 -> 69.2 mm
- net EN5V: track 14.7 -> 15.6 mm
- net BTN_DOWN: track 35.2 -> 34.4 mm
- net EN15V: track 14.7 -> 15.5 mm
- net EN9V: track 15.2 -> 15.9 mm
- net ENOUT: track 91.2 -> 90.6 mm, vias 0 -> 1
Other:
- board size 62 x 53 mm -> 62 x 55.3 mm
- board text added: "By Manuel Mayrhofer and Johannes Melcher-Millner V3.1"
- board text added: "HTL-Rankweil 4AHEL Manuel Mayrhofer Johannes Melcher-Millner PD-LabSupply v3.1 11/23"
- board text removed: "HTL-Rankweil 4AHEL Manuel Mayrhofer Johannes Melcher-Millner USBC_PD-Trigger v3.1 11/23"

Commit message: new version
Parts:
- moved U6 1.96 mm to (83.0, 87.2)

Commit message: layout finished
Parts:
- removed U2: Pico, MCU_RaspberryPi_and_Boards:RPi_Pico_THT
- added C16: 1uF 50v, Capacitor_SMD:C_0805_2012Metric, F.Cu at (120.8, 58.3)
- added C17: 0.1uF, Capacitor_SMD:C_0805_2012Metric, F.Cu at (97.1, 51.9)
- added C18: 27pF, Capacitor_SMD:C_0805_2012Metric, F.Cu at (129.2, 47.9)
- added C19: 27pF, Capacitor_SMD:C_0805_2012Metric, F.Cu at (129.2, 44.4)
- added C20: 0.1uF, Capacitor_SMD:C_0805_2012Metric, F.Cu at (121.3, 43.8)
- added C21: 0.1uF, Capacitor_SMD:C_0805_2012Metric, F.Cu at (105.5, 45.8)
- added C22: 0.1uF, Capacitor_SMD:C_0805_2012Metric, F.Cu at (114.7, 56.9)
- added C23: 0.1uF, Capacitor_SMD:C_0805_2012Metric, F.Cu at (105.5, 53.9)
- added C24: 0.1uF, Capacitor_SMD:C_0805_2012Metric, F.Cu at (121.3, 47.3)
- added C25: 0.1uF, Capacitor_SMD:C_0805_2012Metric, F.Cu at (116.7, 56.9)
- added C26: 0.1uF, Capacitor_SMD:C_0805_2012Metric, F.Cu at (105.5, 51.9)
- added C27: 0.1uF, Capacitor_SMD:C_0805_2012Metric, F.Cu at (105.5, 43.8)
- added C28: 1uF 50v, Capacitor_SMD:C_0805_2012Metric, F.Cu at (109.6, 42.3)
- added C29: 1uF 50v, Capacitor_SMD:C_0805_2012Metric, F.Cu at (111.6, 42.3)
- added C30: 0.1uF, Capacitor_SMD:C_0805_2012Metric, F.Cu at (105.5, 41.7)
- added C8: 1uF 50v, Capacitor_SMD:C_0805_2012Metric, F.Cu at (127.1, 58.3)
- added R13: 10k, Resistor_SMD:R_0805_2012Metric, F.Cu at (118.7, 58.3)
- added R14: 10k, Resistor_SMD:R_0805_2012Metric, F.Cu at (97.1, 55.5)
- added R15: 1k, Resistor_SMD:R_0805_2012Metric, F.Cu at (95.1, 55.5)
- added R17: 10k, Resistor_SMD:R_0805_2012Metric, F.Cu at (131.3, 44.4)
- added R18: 27, Resistor_SMD:R_0805_2012Metric, F.Cu at (105.5, 49.9)
- added R19: 27, Resistor_SMD:R_0805_2012Metric, F.Cu at (105.5, 47.8)
- added R20: DNP, Resistor_SMD:R_0805_2012Metric, F.Cu at (121.3, 54.3)
- added R21: 1K, Resistor_SMD:R_0805_2012Metric, F.Cu at (121.3, 50.9)
- added SW6: SW_Push, Button_Switch_SMD:SW_SPST_TL3305B, F.Cu at (89.3, 54.8)
- added TP1: TestPoint, TestPoint:TestPoint_Pad_D2.0mm, B.Cu at (91.2, 48.2)
- added TP2: TestPoint, TestPoint:TestPoint_Pad_D2.0mm, B.Cu at (91.2, 44.0)
- added TP3: TestPoint, TestPoint:TestPoint_Pad_D2.0mm, B.Cu at (98.3, 56.2)
- added TP4: TestPoint, TestPoint:TestPoint_Pad_D2.0mm, B.Cu at (101.6, 56.3)
- added U5: RP2040, Package_DFN_QFN:QFN-56-1EP_7x7mm_P0.4mm_EP3.2x3.2mm, F.Cu at (114.0, 49.1)
- added U8: AP2112K-3.3TRG1, Package_TO_SOT_SMD:SOT-23-5, F.Cu at (123.9, 58.3)
- added U9: W25Q16JVSSIQ, Package_SO:SOIC-8_3.9x4.9mm_P1.27mm, F.Cu at (100.9, 53.6)
- added XTAL1: ABLS-12.000MHZ-B2-T, ABLS_12_000MHZ_B2_T:XTAL_HC&slash_49US_ABLS_ABR, F.Cu at (125.3, 49.0)
- C10: value 22u 50V -> 22uF 50V
- C14: value 1uF -> 1uF 50V
- C3: value 2.2u 50V -> 2.2uF 50V
- C5: value 0.1u -> 0.1uF
- C9: value 22u -> 22u 50V
- D2, J1, J2, J4, J5, SW2, SW3, SW4, SW5, U6: moved to B.Cu
- J6: footprint Connector_PinSocket_2.54mm:PinSocket_1x07_P2.54mm_Vertical -> Connector_PinSocket_2.54mm:PinSocket_1x07_P2.54mm_Vertical_SMD_Pin1Left; moved to B.Cu
- J7: footprint Connector_PinHeader_2.54mm:PinHeader_1x02_P2.54mm_Vertical -> Connector_PinHeader_2.54mm:PinHeader_1x02_P2.54mm_Horizontal; moved to B.Cu
- J8: value Conn_01x02 -> Conn_02x02_Counter_Clockwise; footprint Connector_PinHeader_2.54mm:PinHeader_1x02_P2.54mm_Vertical -> Connector_PinSocket_2.54mm:PinSocket_2x02_P2.54mm_Horizontal
- L1: value L -> 15uH
- R12, R16: footprint Capacitor_SMD:C_1206_3216Metric -> Resistor_SMD:R_1206_3216Metric
- R2: value 118k -> 120k
- R3: value 22.1k -> 22k
- R5, R7: value 4k7 -> 5k1
- SW1: footprint Button_Switch_THT:SW_DIP_SPSTx06_Slide_9.78x17.42mm_W7.62mm_P2.54mm -> Button_Switch_SMD:SW_DIP_SPSTx06_Slide_9.78x17.42mm_W8.61mm_P2.54mm; moved to B.Cu
- moved U6 54.5 mm to (80.7, 32.7)
- moved SW2 51.0 mm to (113.8, 34.4)
- moved SW5 51.0 mm to (123.8, 34.4)
- moved D2 44.8 mm to (132.6, 35.1), turned to 180 degrees
- moved H3 41.9 mm to (70.2, 40.1)
- moved SW4 41.3 mm to (123.8, 39.7), turned to 180 degrees
- moved SW3 40.6 mm to (113.6, 39.7), turned to 180 degrees
- moved H4 26.7 mm to (139.3, 58.1)
- moved J2 23.5 mm to (155.7, 51.4)
- moved SW1 23.2 mm to (118.4, 49.1), turned to -90 degrees
- moved J4 22.8 mm to (153.2, 47.5), turned to -90 degrees
- moved J5 20.5 mm to (155.7, 55.2)
- moved C7 18.1 mm to (129.9, 41.6), turned to 0 degrees
- moved D1 18.0 mm to (134.5, 43.4)
- moved Q4 18.0 mm to (124.2, 37.8)
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Connections:
- J7 pad 1: CC1 -> SDA
- J7 pad 2: CC2 -> SCL
- J8 pad 1: SCL -> unconnected-(J8-Pin_1-Pad1)
- J8 pad 2: SDA -> unconnected-(J8-Pin_2-Pad2)
- U1 pad 4: D_P -> D_N
- U1 pad 6: D_N -> D_P
Routing:
- net ENOUT: track 90.6 -> 27.5 mm
- net +3V3: track 0.00 -> 62.8 mm, vias 0 -> 4
- net CC2: track 72.7 -> 14.1 mm, vias 3 -> 1
- net CC1: track 69.2 -> 14.5 mm, vias 3 -> 1
- net LED: track 46.6 -> 1.66 mm
- net SW_OUT: track 44.6 -> 0.00 mm
- net BTN_DOWN: track 34.4 -> 0.00 mm
- net SW_VA: track 33.7 -> 0.00 mm
- net VBUS: track 31.9 -> 0.00 mm, vias 9 -> 0
- net SDA: track 71.7 -> 40.4 mm, vias 1 -> 3
- net BTN_UP: track 27.4 -> 0.00 mm
- net XIN: track 0.00 -> 22.3 mm
- net QSPI_SS: track 0.00 -> 21.6 mm
- net OUT: track 20.3 -> 0.00 mm, vias 15 -> 0
- net Net-(Q4-G): track 23.7 -> 4.09 mm, vias 2 -> 0
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- added copper zone on F.Cu, net +3V3
- removed copper zone on B.Cu, net (none)
- removed copper zone on F.Cu, net (none)
- removed copper zone on B.Cu, net +5V
- removed copper zone on F.Cu, net /SW
- removed copper zone on F.Cu, net HALL_IN
- removed copper zone on B.Cu, net OUT
- removed copper zone on F.Cu, net OUT
- removed copper zone on B.Cu, net VBUS
- removed copper zone on F.Cu, net VBUS
Other:
- board size 62 x 55.3 mm -> 62 x 28.8 mm
- board text added: "CC1"
- board text added: "CC2"
- board text added: "Manuel Mayrhofer Johannes Melcher-Millner V4.0"
- board text added: "SCL"
- board text added: "SDA"
- board text removed: "By Manuel Mayrhofer and Johannes Melcher-Millner V3.1"
- board text removed: "CC1 CC2"
- board text removed: "POGOPINS"
- board text removed: "SDA SCL"

Commit message: layout almost complete
Parts:
- added C31: 0.1uF, Capacitor_SMD:C_0805_2012Metric, F.Cu at (105.4, 54.2)
- C21: value 0.1uF -> 1uF 50v
- moved C26 1.81 mm to (105.4, 50.1)
- moved C27 1.81 mm to (105.4, 42.0)
- moved R19 1.81 mm to (105.4, 46.0)
- moved C21 1.81 mm to (105.4, 44.0)
- moved C23 1.81 mm to (105.4, 52.1)
- moved C30 1.81 mm to (105.4, 39.9)
- moved R18 1.81 mm to (105.4, 48.1)
- moved R17 0.89 mm to (132.2, 44.4)
- moved SW1 0.76 mm to (118.2, 48.3)
- moved J6 0.63 mm to (118.4, 57.5)
- moved XTAL1 0.54 mm to (125.3, 48.4)
- moved C1 0.17 mm to (90.4, 51.2)
- moved R1 0.16 mm to (90.4, 49.2)
- moved R3 0.11 mm to (129.2, 51.4)
- moved C9 0.06 mm to (129.2, 58.3)
Routing:
- net +3V3: track 62.8 -> 168.8 mm, vias 4 -> 11
- net +5V: track 0.00 -> 88.5 mm, vias 0 -> 3
- net LED: track 1.66 -> 50.2 mm, vias 0 -> 1
- net ADC0: track 0.00 -> 45.9 mm, vias 0 -> 2
- net VBUS: track 0.00 -> 39.1 mm, vias 0 -> 4
- net SW_VA: track 0.00 -> 38.8 mm, vias 0 -> 1
- net SCL: track 46.4 -> 77.8 mm
- net SDA: track 40.4 -> 71.1 mm
- net SW_OUT: track 0.00 -> 30.5 mm, vias 0 -> 1
- net BTN_DOWN: track 0.00 -> 20.3 mm, vias 0 -> 1
- net /+1.1V: track 12.3 -> 32.2 mm
- net BTN_UP: track 0.00 -> 19.2 mm, vias 0 -> 1
- net VDD: track 0.00 -> 10.1 mm, vias 5 -> 7
- net ENOUT: track 27.5 -> 35.0 mm
- net Net-(U4-V3VD): track 0.00 -> 6.16 mm
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- added copper zone on F.Cu, net (none)
- added copper zone on F.Cu, net /SW
- added copper zone on F.Cu, net HALL_IN
- added copper zone on F.Cu, net OUT
- added copper zone on F.Cu, net VBUS

Commit message: layout finished
Parts:
- removed J2, J4, J5: Conn_01x02, Connector_PinHeader_2.54mm:PinHeader_1x02_P2.54mm_Vertical
- removed J7: Conn_01x02, Connector_PinHeader_2.54mm:PinHeader_1x02_P2.54mm_Horizontal
- moved J8 17.5 mm to (138.0, 53.0)
Connections:
- J8 pad 1: unconnected-(J8-Pin_1-Pad1) -> GND
- J8 pad 2: unconnected-(J8-Pin_2-Pad2) -> SDA
- J8 pad 3: unconnected-(J8-Pin_3-Pad3) -> +5V
- J8 pad 4: unconnected-(J8-Pin_4-Pad4) -> SCL
Routing:
- net OUT: track 0.00 -> 63.7 mm, vias 0 -> 4
- net SDA: track 71.1 -> 83.9 mm, vias 3 -> 4
- net SCL: track 77.8 -> 85.1 mm, vias 3 -> 4
- net +5V: track 88.5 -> 94.2 mm, vias 3 -> 5
- net EN5V: track 11.6 -> 12.6 mm
- net VBUS: track 39.1 -> 38.5 mm
- net GND: vias 18 -> 60

Commit message: save
Routing:
- net Net-(U7-CB): track 0.00 -> 2.16 mm
- net GND: vias 60 -> 61
Changed lines of the file:
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@@
   (via (at 114.56354 47.0825) (size 0.5) (drill 0.25) (layers "F.Cu" "B.Cu") (free) (net 1))
   (via (at 94.755 44.501) (size 0.5) (drill 0.25) (layers "F.Cu" "B.Cu") (free) (net 1))
+  (via (at 100.089 41.199) (size 0.5) (drill 0.25) (layers "F.Cu" "B.Cu") (free) (net 1))
   (via (at 103.645 52.121) (size 0.5) (drill 0.25) (layers "F.Cu" "B.Cu") (free) (net 1))
   (via (at 104.026 42.977) (size 0.5) (drill 0.25) (layers "F.Cu" "B.Cu") (free) (net 1))
@@
   (segment (start 129.172 53.137) (end 130.95 51.359) (width 0.2) (layer "B.Cu") (net 48))
   (segment (start 130.95 51.359) (end 134.887 51.359) (width 0.2) (layer "B.Cu") (net 48))
+  (segment (start 133.858 53.259) (end 134.7855 53.259) (width 0.4) (layer "F.Cu") (net 49))
+  (segment (start 135.3645 53.838) (end 135.776 53.838) (width 0.4) (layer "F.Cu") (net 49))
+  (segment (start 134.7855 53.259) (end 135.3645 53.838) (width 0.4) (layer "F.Cu") (net 49))
   (segment (start 113.646 41.4095) (end 115.308 41.4095) (width 0.2) (layer "F.Cu") (net 50))
   (segment (start 115.308 41.4095) (end 115.49 41.2275) (width 0.2) (layer "F.Cu") (net 50))
