File: PD-LabSupply.kicad_pcb (KiCad board)
At the start: 2 copper layers, 62 x 28.8 mm, 85 parts, among them J1 Conn_01x02, J3 USB_C_Receptacle_USB2.0, J6 Conn_01x07, J8 Conn_02x02_Counter_Clockwise, Q1 BC847, Q4 IRF9393, SW1 SW_DIP_x06, SW2 SW_DPST_x2, SW3 SW_Push, SW4 SW_Push, SW5 SW_DPST_x2, SW6 SW_Push, U1 SRV05-4, U3 TMCS1108, U4 AP33772, U5 RP2040, U6 oledSym, U7 LMR54410, U8 AP2112K-3.3TRG1, U9 W25Q16JVSSIQ

Commit message: save
Parts:
- removed J8: Conn_02x02_Counter_Clockwise, Connector_PinSocket_2.54mm:PinSocket_2x02_P2.54mm_Horizontal
- removed XTAL1: ABLS-12.000MHZ-B2-T, ABLS_12_000MHZ_B2_T:XTAL_HC&slash_49US_ABLS_ABR
- added J2: Conn_02x02_Odd_Even, Connector_PinSocket_2.54mm:PinSocket_2x02_P2.54mm_Horizontal, B.Cu at (131.8, 50.3)
- added SW7: SW_Push, Button_Switch_SMD:SW_SPST_PTS810, B.Cu at (118.8, 39.8)
- added Y1: Crystal_GND24, Crystal:Crystal_SMD_3225-4Pin_3.2x2.5mm, F.Cu at (126.1, 47.8)
- C18, C19: value 27pF -> 15pF
- L1: footprint -Passive:L_4012 -> PCM_Inductor_SMD_AKL:L_Taiyo-Yuden_MD-5050
- SW3, SW4, SW6: footprint Button_Switch_SMD:SW_SPST_TL3305B -> Button_Switch_SMD:SW_SPST_PTS810
- moved C3 14.5 mm to (123.7, 58.7), turned to 90 degrees
- moved C10 11.4 mm to (125.8, 58.7), turned to 90 degrees
- moved C9 8.75 mm to (136.9, 54.3), turned to 0 degrees
- moved C8 7.98 mm to (120.7, 53.6), turned to 0 degrees
- moved U7 7.40 mm to (128.8, 58.6), turned to 90 degrees
- moved R3 6.62 mm to (124.4, 55.9), turned to 180 degrees
- moved C5 6.20 mm to (129.6, 54.9), turned to 90 degrees
- moved R20 4.10 mm to (123.3, 50.8)
- moved R21 4.10 mm to (123.3, 47.3)
- moved U8 3.62 mm to (120.7, 56.7), turned to 90 degrees
- moved R17 3.30 mm to (128.9, 44.4)
- moved C16 3.15 mm to (117.9, 56.9)
- moved C19 3.06 mm to (126.1, 44.6), turned to 0 degrees
- moved R13 2.45 mm to (120.7, 59.8), turned to 0 degrees
- moved SW4 2.16 mm to (126.0, 39.8)
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Connections:
- U5 pad 27: unconnected-(U5-GPIO16-Pad27) -> BTN_SEL
Routing:
- net +5V: track 94.2 -> 129.6 mm, vias 5 -> 6
- net VBUS: track 38.5 -> 18.3 mm, vias 4 -> 6
- net +3V3: track 168.6 -> 151.5 mm, vias 11 -> 9
- net SCL: track 85.1 -> 69.4 mm
- net Net-(C19-Pad1): track 15.6 -> 4.21 mm
- net BTN_SEL: track 0.00 -> 10.8 mm, vias 0 -> 1
- net SDA: track 83.9 -> 74.8 mm
- net XIN: track 22.9 -> 14.2 mm
- net Net-(U5-RUN): track 24.3 -> 18.5 mm
- net Net-(U7-FB): track 9.08 -> 3.84 mm, vias 2 -> 0
- net Net-(R15-Pad1): track 10.5 -> 6.37 mm
- net EN15V: track 12.0 -> 7.91 mm
- net Net-(U8-EN): track 5.90 -> 2.01 mm
- net ENPSU: track 13.4 -> 10.4 mm
- net OUT: track 63.7 -> 62.5 mm
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- added copper zone on B.Cu, net VBUS

Commit message: fertig
Parts:
- removed J3: USB_C_Receptacle_USB2.0, Connector_USB:USB_C_Receptacle_JAE_DX07S016JA1R1500
- added J4: USB4500-03-0-A, USB4500_03_0_A:CONN_USB4500_GCT, B.Cu at (83.4, 46.1)
- L1: footprint PCM_Inductor_SMD_AKL:L_Taiyo-Yuden_MD-5050 -> Inductor_SMD:L_Coilcraft_XAL5050-XXX

Commit message: finished
Parts:
- removed H1, H3: MountingHole, MountingHole:MountingHole_2.5mm
- removed J4: USB4500-03-0-A, USB4500_03_0_A:CONN_USB4500_GCT
- removed Q1: BC847, Package_TO_SOT_SMD:SOT-23
- removed Q4: IRF9393, Package_SO:SOIC-8_3.9x4.9mm_P1.27mm
- removed R5, R7: 5k1, Resistor_SMD:R_0805_2012Metric
- removed R6: 10k, Resistor_SMD:R_0805_2012Metric
- removed R8: 1k, Resistor_SMD:R_0805_2012Metric
- removed SW5: SW_DPST_x2, Button_Switch_SMD:SW_SPDT_PCM12
- added J3: USB4520-03-0-A, USB4520_03_0_A:CONN12_USB4520-03-0-A_GCT, B.Cu at (80.1, 53.1)
- added Q2: DMN3008SFGQ-7, DMN3008SFGQ-7:DMG7401SFG13, F.Cu at (124.2, 37.8)
- added SW8: JS202011JAQN, JS202011JAQN:JS202011JAQN, B.Cu at (124.2, 33.5)
- L1: footprint Inductor_SMD:L_Coilcraft_XAL5050-XXX -> Inductor_SMD:L_Taiyo-Yuden_MD-5050
- SW2: value SW_DPST_x2 -> JS202011JAQN; footprint Button_Switch_SMD:SW_SPDT_PCM12 -> JS202011JAQN:JS202011JAQN
- U3: footprint Package_SO:SOIC-8_3.9x4.9mm_P1.27mm -> PCM_4ms_Package_SOIC:SOIC-8_3.9x4.9mm_Pitch1.27mm
- U4: footprint Package_DFN_QFN:WQFN-24-1EP_4x4mm_P0.5mm_EP2.6x2.6mm_ThermalVias -> AP33772:AP33772
- U8: footprint Package_TO_SOT_SMD:SOT-23-5 -> AP2112K_3_3TRG1:SOT_RG1_DIO
- moved C1 1.19 mm to (90.4, 52.4)
- moved R1 1.19 mm to (90.4, 50.4)
- moved SW2 1.04 mm to (113.8, 33.4)
- moved C18 0.13 mm to (128.9, 47.9)
- moved C14 0.10 mm to (97.9, 48.7)
- moved U8 0.08 mm to (120.8, 56.7)
Connections:
- net /SHIELD renamed Net-(C1-Pad1)
- J6 pad 2: ENOUT -> EXT_OUT
- SW2 pad 1: GND -> SW_VA
- SW2 pad 2: SW_OUT -> SW_VA
- SW2 pad 3: (no net) -> GND
- U4 pad 23: unconnected-(U4-PWR_EN-Pad23) -> ENOUT
- U5 pad 15: SW_OUT -> EXT_OUT
- U5 pad 16: SW_VA -> unconnected-(U5-GPIO13-Pad16)
- U5 pad 17: BTN_DOWN -> unconnected-(U5-GPIO14-Pad17)
- U5 pad 18: BTN_UP -> unconnected-(U5-GPIO15-Pad18)
- U5 pad 27: BTN_SEL -> unconnected-(U5-GPIO16-Pad27)
- U5 pad 29: unconnected-(U5-GPIO18-Pad29) -> BTN_DOWN
- U5 pad 30: unconnected-(U5-GPIO19-Pad30) -> BTN_SEL
- U5 pad 31: unconnected-(U5-GPIO20-Pad31) -> BTN_UP
- U5 pad 32: ENOUT -> SW_VA
- U5 pad 34: unconnected-(U5-GPIO22-Pad34) -> LED
- U5 pad 35: unconnected-(U5-GPIO23-Pad35) -> SW_OUT
- U5 pad 38: ADC0 -> unconnected-(U5-GPIO26_ADC0-Pad38)
- U5 pad 41: unconnected-(U5-GPIO29_ADC3-Pad41) -> ADC0
- U5 pad 5: LED -> unconnected-(U5-GPIO3-Pad5)
Routing:
- net SW_VA: track 38.3 -> 13.9 mm
- net EXT_OUT: track 0.00 -> 19.9 mm, vias 0 -> 1
- net LED: track 49.0 -> 32.8 mm
- net ADC0: track 44.6 -> 29.9 mm
- net SW_OUT: track 30.4 -> 22.2 mm
- net BTN_UP: track 18.5 -> 10.3 mm
- net +3V3: track 151.5 -> 144.7 mm, vias 9 -> 10
- net Net-(Q1-C): track 6.04 -> 0.00 mm
- net GND: track 4.48 -> 0.31 mm, vias 68 -> 72
- net Net-(Q4-G): track 4.09 -> 0.00 mm
- net Net-(Q1-B): track 4.05 -> 0.00 mm
- net BTN_DOWN: track 21.4 -> 17.6 mm
- net SCL: track 69.4 -> 72.4 mm
- net ENOUT: track 35.0 -> 33.0 mm, vias 1 -> 2
- net VDD: track 10.1 -> 8.75 mm, vias 7 -> 4
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Other:
- outline, holes or cut-outs redrawn
- board text added: "HTL-Rankweil 4AHEL Manuel Mayrhofer Johannes Melcher-Millner PD-LabSupply v4.2 12/23"
- board text added: "Manuel Mayrhofer Johannes Melcher-Millner V4.2"
- board text removed: "HTL-Rankweil 4AHEL Manuel Mayrhofer Johannes Melcher-Millner PD-LabSupply v3.1 11/23"
- board text removed: "Manuel Mayrhofer Johannes Melcher-Millner V4.0"
