File: PD-LabSupply.kicad_pcb (KiCad board)
At the start: 2 copper layers, 62 x 28.8 mm, 79 parts, among them J1 Conn_01x02, J2 Conn_02x02_Odd_Even, J3 USB4520-03-0-A, J6 Conn_01x07, Q2 DMN3008SFGQ-7, SW1 SW_DIP_x06, SW2 JS202011JAQN, SW3 SW_Push, SW4 SW_Push, SW6 SW_Push, SW7 SW_Push, SW8 JS202011JAQN, U1 SRV05-4, U3 TMCS1108, U4 AP33772, U5 RP2040, U6 oledSym, U7 LMR54410, U8 AP2112K-3.3TRG1, U9 W25Q16JVSSIQ, Y1 Crystal_GND24

Commit message: wirklich mol fertig
Other:
- board text removed: "+5V"
- board text removed: "12V"
- board text removed: "15V"
- board text removed: "20V"
- board text removed: "5V"
- board text removed: "9V"
- board text removed: "CHANGE"
- board text removed: "DOWN"
- board text removed: "ENABLE OUTPUT"
- board text removed: "Max A"
- board text removed: "OFF"
- board text removed: "ON"
- board text removed: "PPS"
- board text removed: "UP"
- board text removed: "V"

Commit message: bestellung
Routing:
- net GND: vias 72 -> 71

Commit message: changes
Parts:
- added R5: 1k, Resistor_SMD:R_0805_2012Metric, F.Cu at (123.3, 43.8)
Connections:
- Q2 pad G: ENOUT -> Net-(Q2-PadG)
Routing:
- net ENOUT: track 33.0 -> 27.7 mm
- net Net-(Q2-PadG): track 0.00 -> 4.25 mm
Changed lines of the file:
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@@
   (net 86 "unconnected-(SW8-Pad6)")
   (net 87 "unconnected-(SW8-Pad7)")
+  (net 88 "Net-(Q2-PadG)")
   (footprint "Crystal:Crystal_SMD_3225-4Pin_3.2x2.5mm" (layer "F.Cu")
     (at 126.124 47.803 90)
@@
     )
   )
+  (footprint "Resistor_SMD:R_0805_2012Metric" (layer "F.Cu")
+    (at 123.33 43.7625 90)
+    (descr "Resistor SMD 0805 (2012 Metric), square (rectangular) end terminal, IPC_7351 nominal, (Body size source: IPC-SM-782 page 72, https://www.pcb-3d.com/wordpress/wp-content/uploads/ipc-sm-782a_amendment_1_and_2.pdf), generated with kicad-footprint-generator")
+    (tags "resistor")
+    (property "Sheetfile" "PD-LabSupply.kicad_sch")
+    (property "Sheetname" "")
+    (attr smd)
+    (fp_text reference "R5" (at 0 -1.65 90) (layer "F.SilkS")
+        (effects (font (size 1 1) (thickness 0.15)))
+    )
+    (fp_text value "1k" (at 0 1.65 90) (layer "F.Fab")
+        (effects (font (size 1 1) (thickness 0.15)))
+    )
+    (fp_text user "${REFERENCE}" (at 0 0 90) (layer "F.Fab")
+        (effects (font (size 0.5 0.5) (thickness 0.08)))
+    )
+    (fp_line (start -0.227064 -0.735) (end 0.227064 -0.735)
+      (stroke (width 0.12) (type solid)) (layer "F.SilkS"))
+    (fp_line (start -0.227064 0.735) (end 0.227064 0.735)
+      (stroke (width 0.12) (type solid)) (layer "F.SilkS"))
+    (fp_line (start -1.68 -0.95) (end 1.68 -0.95)
+      (stroke (width 0.05) (type solid)) (layer "F.CrtYd"))
+    (fp_line (start -1.68 0.95) (end -1.68 -0.95)
+      (stroke (width 0.05) (type solid)) (layer "F.CrtYd"))
+    (fp_line (start 1.68 -0.95) (end 1.68 0.95)
+      (stroke (width 0.05) (type solid)) (layer "F.CrtYd"))
+    (fp_line (start 1.68 0.95) (end -1.68 0.95)
+      (stroke (width 0.05) (type solid)) (layer "F.CrtYd"))
+    (fp_line (start -1 -0.625) (end 1 -0.625)
+      (stroke (width 0.1) (type solid)) (layer "F.Fab"))
+    (fp_line (start -1 0.625) (end -1 -0.625)
+      (stroke (width 0.1) (type solid)) (layer "F.Fab"))
+    (fp_line (start 1 -0.625) (end 1 0.625)
+      (stroke (width 0.1) (type solid)) (layer "F.Fab"))
+    (fp_line (start 1 0.625) (end -1 0.625)
+      (stroke (width 0.1) (type solid)) (layer "F.Fab"))
+    (pad "1" smd roundrect (at -0.9125 0 90) (size 1.025 1.4) (layers "F.Cu" "F.Paste" "F.Mask") (roundrect_rratio 0.243902)
+      (net 6 "ENOUT") (pintype "passive"))
+    (pad "2" smd roundrect (at 0.9125 0 90) (size 1.025 1.4) (layers "F.Cu" "F.Paste" "F.Mask") (roundrect_rratio 0.243902)
+      (net 88 "Net-(Q2-PadG)") (pintype "passive"))
+    (model "${KICAD6_3DMODEL_DIR}/Resistor_SMD.3dshapes/R_0805_2012Metric.wrl"
+      (offset (xyz 0 0 0))
+      (scale (xyz 1 1 1))
+      (rotate (xyz 0 0 0))
+    )
+  )
   (footprint "Capacitor_SMD:C_0805_2012Metric" (layer "F.Cu")
     (at 129.934 41.56)
@@
       (net 2 "HALL_IN") (pinfunction "D") (pintype "passive"))
     (pad "G" smd rect (at 0.975 1.35 270) (size 0.42 0.7) (layers "F.Cu" "F.Paste" "F.Mask")
-      (net 6 "ENOUT") (pinfunction "G") (pintype "passive"))
+      (net 88 "Net-(Q2-PadG)") (pinfunction "G") (pintype "passive"))
     (pad "S" smd rect (at -0.975 1.35 270) (size 0.42 0.7) (layers "F.Cu" "F.Paste" "F.Mask")
       (net 5 "VBUS") (pinfunction "S") (pintype "passive"))
@@
   (via (at 96.152 55.423) (size 0.5) (drill 0.25) (layers "F.Cu" "B.Cu") (free) (net 1))
   (via (at 103.518 49.708) (size 0.5) (drill 0.25) (layers "F.Cu" "B.Cu") (free) (net 1))
-  (via (at 123.2538 42.6468) (size 0.5) (drill 0.25) (layers "F.Cu" "B.Cu") (free) (net 1))
+  (via (at 125.4636 42.0372) (size 0.5) (drill 0.25) (layers "F.Cu" "B.Cu") (free) (net 1))
   (via (at 125.4636 54.0768) (size 0.5) (drill 0.25) (layers "F.Cu" "B.Cu") (free) (net 1))
   (via (at 131.9406 45.2376) (size 0.5) (drill 0.25) (layers "F.Cu" "B.Cu") (free) (net 1))
@@
   (via (at 128.41 54.9404) (size 0.5) (drill 0.25) (layers "F.Cu" "B.Cu") (free) (net 1))
   (via (at 112.5096 57.328) (size 0.5) (drill 0.25) (layers "F.Cu" "B.Cu") (free) (net 1))
-  (via (at 123.2538 43.2564) (size 0.5) (drill 0.25) (layers "F.Cu" "B.Cu") (free) (net 1))
+  (via (at 125.4636 42.7484) (size 0.5) (drill 0.25) (layers "F.Cu" "B.Cu") (free) (net 1))
   (via (at 85.6872 38.532) (size 0.5) (drill 0.25) (layers "F.Cu" "B.Cu") (free) (net 1))
   (via (at 131.3818 35.23) (size 0.5) (drill 0.25) (layers "F.Cu" "B.Cu") (free) (net 1))
@@
   (via (at 130.2896 48.2348) (size 0.5) (drill 0.25) (layers "F.Cu" "B.Cu") (free) (net 1))
   (via (at 114.56354 47.0825) (size 0.5) (drill 0.25) (layers "F.Cu" "B.Cu") (free) (net 1))
-  (via (at 123.2538 42.088) (size 0.5) (drill 0.25) (layers "F.Cu" "B.Cu") (free) (net 1))
+  (via (at 124.7524 42.0372) (size 0.5) (drill 0.25) (layers "F.Cu" "B.Cu") (free) (net 1))
   (via (at 123.4316 34.341) (size 0.5) (drill 0.25) (layers "F.Cu" "B.Cu") (free) (net 1))
   (via (at 132.5756 45.2376) (size 0.5) (drill 0.25) (layers "F.Cu" "B.Cu") (free) (net 1))
@@
   (segment (start 97.8284 38.2526) (end 98.3618 37.7192) (width 0.2) (layer "B.Cu") (net 5))
   (segment (start 100.590505 48.101305) (end 101.0796 48.101305) (width 0.2) (layer "F.Cu") (net 6))
-  (segment (start 122.341 45.611986) (end 122.341 41.7562) (width 0.3) (layer "F.Cu") (net 6))
-  (segment (start 122.8944 41.2028) (end 122.8944 38.7804) (width 0.3) (layer "F.Cu") (net 6))
+  (segment (start 123.2792 45.4545) (end 123.2792 44.7258) (width 0.3) (layer "F.Cu") (net 6))
+  (segment (start 123.2792 44.7258) (end 123.33 44.675) (width 0.3) (layer "F.Cu") (net 6))
   (segment (start 100.4255 46.9665) (end 100.4255 47.9363) (width 0.2) (layer "F.Cu") (net 6))
-  (segment (start 122.341 45.611986) (end 122.291 45.661986) (width 0.2) (layer "F.Cu") (net 6))
   (segment (start 100.4255 47.9363) (end 100.590505 48.101305) (width 0.2) (layer "F.Cu") (net 6))
-  (segment (start 122.341 41.7562) (end 122.8944 41.2028) (width 0.3) (layer "F.Cu") (net 6))
   (via (at 101.0796 48.101305) (size 0.5) (drill 0.25) (layers "F.Cu" "B.Cu") (net 6))
-  (via (at 122.341 45.611986) (size 0.5) (drill 0.25) (layers "F.Cu" "B.Cu") (net 6))
-  (segment (start 107.4296 47.6252) (end 107.4138 47.641) (width 0.3) (layer "B.Cu") (net 6))
-  (segment (start 101.539905 47.641) (end 101.0796 48.101305) (width 0.3) (layer "B.Cu") (net 6))
+  (via (at 123.2792 45.4545) (size 0.5) (drill 0.25) (layers "F.Cu" "B.Cu") (net 6))
+  (segment (start 123.2792 45.4545) (end 123.2577 45.476) (width 0.3) (layer "B.Cu") (net 6))
+  (segment (start 123.2577 45.476) (end 118.9768 45.476) (width 0.3) (layer "B.Cu") (net 6))
   (segment (start 107.4138 47.641) (end 101.539905 47.641) (width 0.3) (layer "B.Cu") (net 6))
-  (segment (start 109.7514 49.947) (end 107.4296 47.6252) (width 0.3) (layer "B.Cu") (net 6))
-  (segment (start 122.341 45.611986) (end 118.840814 45.611986) (width 0.3) (layer "B.Cu") (net 6))
-  (segment (start 114.5058 49.947) (end 109.7514 49.947) (width 0.3) (layer "B.Cu") (net 6))
-  (segment (start 118.840814 45.611986) (end 114.5058 49.947) (width 0.3) (layer "B.Cu") (net 6))
+  (segment (start 109.7198 49.947) (end 107.4138 47.641) (width 0.3) (layer "B.Cu") (net 6))
+  (segment (start 101.539905 47.641) (end 101.0796 48.101305) (width 0.3) (layer "B.Cu") (net 6))
+  (segment (start 118.9768 45.476) (end 114.5058 49.947) (width 0.3) (layer "B.Cu") (net 6))
+  (segment (start 114.5058 49.947) (end 109.7198 49.947) (width 0.3) (layer "B.Cu") (net 6))
   (segment (start 113.3224 54.9912) (end 112.9668 54.6356) (width 0.2) (layer "F.Cu") (net 7))
   (segment (start 111.717592 48.316489) (end 111.717592 50.197408) (width 0.2) (layer "F.Cu") (net 7))
@@
   (segment (start 108.782 52.560372) (end 108.782 54.026686) (width 0.2) (layer "F.Cu") (net 80))
   (segment (start 100.311 57.55) (end 100.311 56.038) (width 0.2) (layer "F.Cu") (net 80))
+  (segment (start 122.8944 38.7804) (end 122.8944 39.5188) (width 0.3) (layer "F.Cu") (net 88))
+  (segment (start 122.8944 39.5188) (end 123.33 39.9544) (width 0.3) (layer "F.Cu") (net 88))
+  (segment (start 123.33 39.9544) (end 123.33 42.85) (width 0.3) (layer "F.Cu") (net 88))
   (zone (net 70) (net_name "Net-(C1-Pad1)") (layer "F.Cu") (hatch edge 0.508)
     (priority 1)

Commit message: finished
Parts:
- removed J6: Conn_01x07, Connector_PinSocket_2.54mm:PinSocket_1x07_P2.54mm_Vertical_SMD_Pin1Left
- added R6: X, Resistor_SMD:R_0805_2012Metric, F.Cu at (120.0, 41.0)
- added R7: X, Resistor_SMD:R_0805_2012Metric, F.Cu at (119.2, 43.8)
- added TP10: TestPoint, TestPoint:TestPoint_Pad_D1.5mm, B.Cu at (118.9, 55.9)
- added TP11: TestPoint, TestPoint:TestPoint_Pad_D1.5mm, B.Cu at (114.0, 56.5)
- added TP12: TestPoint, TestPoint:TestPoint_Pad_D1.5mm, B.Cu at (111.4, 56.8)
- added TP13: TestPoint, TestPoint:TestPoint_Pad_D1.5mm, B.Cu at (108.9, 56.1)
- added TP7: TestPoint, TestPoint:TestPoint_Pad_D1.5mm, B.Cu at (123.9, 56.5)
- added TP8: TestPoint, TestPoint:TestPoint_Pad_D1.5mm, B.Cu at (116.5, 56.9)
- added TP9: TestPoint, TestPoint:TestPoint_Pad_D1.5mm, B.Cu at (121.5, 55.4)
- C16, C21, C28, C29, C8: value 1uF 50v -> 1uF 50V
- C18, C19: value 15pF -> 18pF
- C9: value 22u 50V -> 22uF 50V
- TP1, TP2, TP3, TP4: footprint TestPoint:TestPoint_Pad_D2.0mm -> TestPoint:TestPoint_Pad_D1.5mm
- moved Q2 0.24 mm to (124.5, 37.7), turned to 90 degrees
Connections:
- Q2 pad D: HALL_IN -> VBUS
- Q2 pad S: VBUS -> HALL_IN
- U3 pad 7: ADC0 -> HALL_ADC
- U5 pad 40: unconnected-(U5-GPIO28_ADC2-Pad40) -> HALL_ADC
- U5 pad 41: ADC0 -> V_ADC
Routing:
- net ADC0: track 29.9 -> 0.00 mm, vias 2 -> 0
- net HALL_ADC: track 0.00 -> 29.5 mm, vias 0 -> 2
- net V_ADC: track 0.00 -> 14.2 mm, vias 0 -> 2
- net EXT_OUT: track 19.9 -> 6.79 mm
- net +5V: track 129.6 -> 122.3 mm
- net EN20V: track 15.1 -> 10.6 mm
- net Net-(Q2-PadG): track 4.25 -> 8.25 mm
- net EN5V: track 12.6 -> 10.0 mm
- net EN9V: track 5.45 -> 7.81 mm
- net VBUS: track 19.0 -> 21.3 mm
- net EN12V: track 9.57 -> 8.19 mm
- net BTN_SEL: track 11.2 -> 10.0 mm
- net +3V3: track 144.7 -> 144.1 mm
- net GND: vias 71 -> 74
