File: PD-LabSupply.kicad_sch (KiCad schematic)
At the start: 56 parts, among them J1 Conn_01x02, J2 Conn_01x02, J3 USB_C_Receptacle_USB2.0, J4 Conn_01x02, J5 Conn_01x02, J6 Conn_01x07, J7 Conn_01x02, J8 Conn_01x02, Q1 BC847, Q4 IRF9393, SW1 SW_DIP_x06, SW2 SW_DPST_x2, SW3 SW_Push, SW4 SW_Push, SW5 SW_DPST_x2, U1 SRV05-4, U2 Pico, U3 TMCS1108, U4 AP33772, U6 oledSym, U7 LMR54410

Commit message: final
Other:
- note added: "PowerDelivery IC"
- note added: "RGB LED"
- note removed: "LED"
- note removed: "PoverDelivery IC"
- moved on the sheet: H1, H2, H3, H4

Commit message: fine
Parts:
- H1, H2, H3, H4: footprint -Hole:D1_8_PAD -> MountingHole:MountingHole_2.5mm
- U2: footprint MCU_RaspberryPi_and_Boards:RPi_Pico_SMD_TH -> MCU_RaspberryPi_and_Boards:RPi_Pico_THT
- U6: footprint SSD1306:128x64OLED -> SSD1306:SSD1306_0.96_Oled
Other:
- title: USBC_PD-Trigger -> PD-LabSupply
Changed lines of the file:
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@@
   (paper "A4")
   (title_block
-    (title "USBC_PD-Trigger")
+    (title "PD-LabSupply")
     (date "2023-11-26")
     (rev "3.1")
@@
       (effects (font (size 1.27 1.27)) (justify left))
     )
-    (property "Footprint" "-Hole:D1_8_PAD" (at 148.59 170.18 0)
+    (property "Footprint" "MountingHole:MountingHole_2.5mm" (at 148.59 170.18 0)
       (effects (font (size 1.27 1.27)) hide)
     )
@@
       (effects (font (size 1.27 1.27)) (justify left))
     )
-    (property "Footprint" "-Hole:D1_8_PAD" (at 125.73 170.18 0)
+    (property "Footprint" "MountingHole:MountingHole_2.5mm" (at 125.73 170.18 0)
       (effects (font (size 1.27 1.27)) hide)
     )
@@
       (effects (font (size 1.27 1.27)) (justify left))
     )
-    (property "Footprint" "-Hole:D1_8_PAD" (at 148.59 181.61 0)
+    (property "Footprint" "MountingHole:MountingHole_2.5mm" (at 148.59 181.61 0)
       (effects (font (size 1.27 1.27)) hide)
     )
@@
       (effects (font (size 1.27 1.27)) (justify left))
     )
-    (property "Footprint" "-Hole:D1_8_PAD" (at 125.73 181.61 0)
+    (property "Footprint" "MountingHole:MountingHole_2.5mm" (at 125.73 181.61 0)
       (effects (font (size 1.27 1.27)) hide)
     )
@@
       (effects (font (size 1.27 1.27)) (justify left))
     )
-    (property "Footprint" "SSD1306:128x64OLED" (at 265.43 137.16 0)
+    (property "Footprint" "SSD1306:SSD1306_0.96_Oled" (at 265.43 137.16 0)
       (effects (font (size 1.27 1.27)) hide)
     )
@@
       (effects (font (size 1.27 1.27)))
     )
-    (property "Footprint" "MCU_RaspberryPi_and_Boards:RPi_Pico_SMD_TH" (at 179.07 52.07 90)
-      (effects (font (size 1.27 1.27)) hide)
-    )
+    (property "Footprint" "MCU_RaspberryPi_and_Boards:RPi_Pico_THT" (at 179.07 52.07 90)
+      (effects (font (size 1.27 1.27)) hide)
+    )

Commit message: new version
Parts:
- C10: value 22u 50V -> 22uF 50V
- C14: value 1uF -> 1uF 50V
- C3: value 2.2u 50V -> 2.2uF 50V
- C5: value 0.1u -> 0.1uF
- C9: value 22u -> 22u 50V
- L1: value L -> 15uH
- R2: value 118k -> 120k
- R3: value 22.1k -> 22k
- R5, R7: value 4k7 -> 5k1
Changed lines of the file:
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@@
       (effects (font (size 1.27 1.27)) (justify left))
     )
-    (property "Value" "1uF" (at 121.92 105.41 0)
+    (property "Value" "1uF 50V" (at 128.27 105.41 0)
       (effects (font (size 1.016 1.016)) (justify left))
     )
@@
       (effects (font (size 1.27 1.27)))
     )
-    (property "Value" "4k7" (at 204.47 146.05 90)
+    (property "Value" "5k1" (at 204.47 146.05 90)
       (effects (font (size 1.016 1.016)))
     )
@@
   (symbol (lib_id "-Passive:L") (at 115.57 64.77 0) (unit 1)
     (in_bom yes) (on_board yes) (dnp no)
-    (property "Reference" "L1" (at 113.03 67.31 0)
-      (effects (font (size 1.27 1.27)))
-    )
-    (property "Value" "L" (at 115.57 66.04 0)
+    (property "Reference" "L1" (at 115.57 62.23 0)
+      (effects (font (size 1.27 1.27)))
+    )
+    (property "Value" "15uH" (at 119.38 62.23 0)
       (effects (font (size 1.27 1.27)))
     )
@@
       (effects (font (size 1.27 1.27)) (justify left))
     )
-    (property "Value" "22u 50V" (at 73.66 66.04 0)
+    (property "Value" "22uF 50V" (at 73.66 66.04 0)
       (effects (font (size 1.016 1.016)) (justify left))
     )
@@
       (effects (font (size 1.27 1.27)) (justify left))
     )
-    (property "Value" "2.2u 50V" (at 87.63 67.31 0)
+    (property "Value" "2.2uF 50V" (at 87.63 67.31 0)
       (effects (font (size 1.016 1.016)) (justify left))
     )
@@
   )
   (symbol (lib_id "-Passive:C") (at 110.49 60.96 0) (unit 1)
-    (in_bom yes) (on_board yes) (dnp no) (fields_autoplaced)
-    (property "Reference" "C5" (at 113.03 59.6963 0)
-      (effects (font (size 1.27 1.27)) (justify left))
-    )
-    (property "Value" "0.1u" (at 113.03 62.2363 0)
+    (in_bom yes) (on_board yes) (dnp no)
+    (property "Reference" "C5" (at 111.76 55.88 0)
+      (effects (font (size 1.27 1.27)) (justify left))
+    )
+    (property "Value" "0.1uF" (at 111.76 58.42 0)
       (effects (font (size 1.016 1.016)) (justify left))
     )
@@
       (effects (font (size 1.27 1.27)) (justify left))
     )
-    (property "Value" "22.1k" (at 115.57 78.74 0)
+    (property "Value" "22k" (at 115.57 78.74 0)
       (effects (font (size 1.016 1.016)) (justify left))
     )
@@
       (effects (font (size 1.27 1.27)) (justify left))
     )
-    (property "Value" "118k" (at 116.84 71.12 0)
+    (property "Value" "120k" (at 116.84 71.12 0)
       (effects (font (size 1.016 1.016)) (justify left))
     )
@@
       (effects (font (size 1.27 1.27)) (justify left))
     )
-    (property "Value" "22u" (at 129.54 69.8563 0)
+    (property "Value" "22u 50V" (at 129.54 69.8563 0)
       (effects (font (size 1.016 1.016)) (justify left))
     )
@@
       (effects (font (size 1.27 1.27)))
     )
-    (property "Value" "4k7" (at 213.36 130.81 90)
+    (property "Value" "5k1" (at 213.36 130.81 90)
       (effects (font (size 1.016 1.016)))
     )

Commit message: layout finished
Parts:
- removed J8: Conn_01x02, Connector_PinHeader_2.54mm:PinHeader_1x02_P2.54mm_Vertical, symbol -Connector:Conn_01x02
- removed U2: Pico, MCU_RaspberryPi_and_Boards:RPi_Pico_THT, symbol MCU_RaspberryPi_and_Boards:Pico
- added C1, C11, C2, C3, C4, C5, C7, C9: 0.1uF, Capacitor_SMD:C_0805_2012Metric, symbol Device:C
- added C13, C15: 27pF, Capacitor_SMD:C_0805_2012Metric, symbol Device:C
- added C16, C28, C29, C8: 1uF 50v, Capacitor_SMD:C_0805_2012Metric, symbol -Passive:C
- added C17, C30: 0.1uF, Capacitor_SMD:C_0805_2012Metric, symbol -Passive:C
- added J8: Conn_02x02_Counter_Clockwise, Connector_PinSocket_2.54mm:PinSocket_2x02_P2.54mm_Horizontal, symbol Connector_Generic:Conn_02x02_Counter_Clockwise
- added R13, R14, R17: 10k, Resistor_SMD:R_0805_2012Metric, symbol -Passive:R
- added R15: 1k, Resistor_SMD:R_0805_2012Metric, symbol -Passive:R
- added R4 (x2): 27, Resistor_SMD:R_0805_2012Metric, symbol Device:R
- added R6: DNP, Resistor_SMD:R_0805_2012Metric, symbol Device:R
- added R7: 1K, Resistor_SMD:R_0805_2012Metric, symbol Device:R
- added SW6: SW_Push, Button_Switch_SMD:SW_SPST_TL3305B, symbol Switch:SW_Push
- added TP1, TP2, TP3, TP4: TestPoint, TestPoint:TestPoint_Pad_D2.0mm, symbol -Connector:TestPoint
- added U5: RP2040, Package_DFN_QFN:QFN-56-1EP_7x7mm_P0.4mm_EP3.2x3.2mm, symbol MCU_RaspberryPi:RP2040
- added U8: AP2112K-3.3TRG1, Package_TO_SOT_SMD:SOT-23-5, symbol AP2112K_3_3TRG1:AP2112K-3.3TRG1
- added U9: W25Q16JVSSIQ, Package_SO:SOIC-8_3.9x4.9mm_P1.27mm, symbol W25Q16JVSSIQ:W25Q16JVSSIQ
- added XTAL1: ABLS-12.000MHZ-B2-T, ABLS_12_000MHZ_B2_T:XTAL_HC&slash_49US_ABLS_ABR, symbol ABLS_12_000MHZ_B2_T:ABLS-12.000MHZ-B2-T
- J6: footprint Connector_PinSocket_2.54mm:PinSocket_1x07_P2.54mm_Vertical -> Connector_PinSocket_2.54mm:PinSocket_1x07_P2.54mm_Vertical_SMD_Pin1Left
- J7: footprint Connector_PinHeader_2.54mm:PinHeader_1x02_P2.54mm_Vertical -> Connector_PinHeader_2.54mm:PinHeader_1x02_P2.54mm_Horizontal
- R12, R16: footprint Capacitor_SMD:C_1206_3216Metric -> Resistor_SMD:R_1206_3216Metric
- SW1: footprint Button_Switch_THT:SW_DIP_SPSTx06_Slide_9.78x17.42mm_W7.62mm_P2.54mm -> Button_Switch_SMD:SW_DIP_SPSTx06_Slide_9.78x17.42mm_W8.61mm_P2.54mm
Connections:
- net +5V: now also C16.1, R13.1, U8.1 (VIN)
- net ADC0: now also U5.38 (GPIO26_ADC0)
- net BTN_DOWN: now also U5.17 (GPIO14)
- net BTN_UP: now also U5.18 (GPIO15)
- net CC1: now also TP1.1; no longer J7.1 (Pin_1)
- net CC2: now also TP2.1; no longer J7.2 (Pin_2)
- net D_N: now also U1.4 (IO3), R4.2; no longer U1.6 (IO4)
- net D_P: now also U1.6 (IO4), R4.1; no longer U1.4 (IO3)
- net EN12V: now also U5.11 (GPIO8)
- net EN15V: now also U5.12 (GPIO9)
- net EN20V: now also U5.13 (GPIO10)
- net EN5V: now also U5.8 (GPIO6)
- net EN9V: now also U5.9 (GPIO7)
- net ENOUT: now also U5.32 (GPIO21)
- net ENPSU: now also U5.14 (GPIO11)
- net GND: now also C1.2, C11.2, C13.2, C15.2, C16.2, C17.2, C2.2, C28.2, C29.2, C3.2, C30.2, C4.2, C5.2, C7.2, C8.2, C9.2, SW6.1, U5.57 (GND), U8.2 (GND), U9.4 (GND)
- net LED: now also U5.5 (GPIO3)
- net SCL: now also J7.2 (Pin_2), TP4.1, U5.7 (GPIO5)
- net SDA: now also J7.1 (Pin_1), TP3.1, U5.6 (GPIO4)
- net SW_OUT: now also U5.15 (GPIO12)
- net SW_VA: now also U5.16 (GPIO13)
- new net: R17.2, U5.26 (RUN)
- new net: R13.2, U8.3 (EN)
- new net: C15.1, R7.2, XTAL1.2
- new net: R15.1, SW6.2
- new net: R4.1, U5.46 (USB_DM)
- new net: R4.2, U5.47 (USB_DP)
- new net +1.1V: C11.1, C9.1, U5.23 (DVDD), U5.45 (VREG_VOUT), U5.50 (DVDD)
- new net +3V3: C1.1, C17.1, C2.1, C28.1, C29.1, C3.1, C30.1, C4.1, C5.1, C7.1, C8.1, R14.1, R17.1, U5.1 (IOVDD), U5.10 (IOVDD), U5.22 (IOVDD), U5.33 (IOVDD), U5.42 (IOVDD), U5.43 (ADC_AVDD), U5.44 (VREG_IN), U5.48 (USB_VDD), U5.49 (IOVDD), U8.5 (VOUT), U9.8 (VCC)
- new net QSPI_SCLK: U5.52 (QSPI_SCLK), U9.6 (CLK)
- new net QSPI_SD0: U5.53 (QSPI_SD0), U9.5 (DI(IO0))
- new net QSPI_SD1: U5.55 (QSPI_SD1), U9.2 (DO(IO1))
- new net QSPI_SD2: U5.54 (QSPI_SD2), U9.3 (~{WP}(IO2))
- new net QSPI_SD3: U5.51 (QSPI_SD3), U9.7 (~{HOLD/RESET}(IO3))
- new net QSPI_SS: R14.2, R15.2, U5.56 (QSPI_SS), U9.1 (~{CS})
- new net XIN: C13.1, R6.2, U5.20 (XIN), XTAL1.1
- new net XOUT: R6.1, R7.1, U5.21 (XOUT)
- no-connect marks 3 -> 4
Other:
- note added: "Each close to an IOVDD pin"

Commit message: layout almost complete
Parts:
- added C11: 0.1uF, Capacitor_SMD:C_0805_2012Metric, symbol Device:C
- C11: value 0.1uF -> 1uF 50v
Connections:
- net +1.1V: now also C11.1
- net GND: now also C11.2
Other:
- moved on the sheet: C11, C9
Changed lines of the file:
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@@
   (junction (at 434.34 -1.27) (diameter 0) (color 0 0 0 0)
   )
+  (junction (at 336.55 -5.08) (diameter 0) (color 0 0 0 0)
+  )
   (junction (at 361.95 -2.54) (diameter 0) (color 0 0 0 0)
   )
@@
   (junction (at 25.4 97.79) (diameter 0) (color 0 0 0 0)
   )
+  (junction (at 342.9 -5.08) (diameter 0) (color 0 0 0 0)
+  )
   (junction (at 25.4 95.25) (diameter 0) (color 0 0 0 0)
   )
@@
   (junction (at 87.63 60.96) (diameter 0) (color 0 0 0 0)
   )
-  (junction (at 337.82 -5.08) (diameter 0) (color 0 0 0 0)
-  )
   (junction (at 121.92 72.39) (diameter 0) (color 0 0 0 0)
   )
@@
     (stroke (width 0) (type default))
   )
-  (wire (pts (xy 331.47 -3.81) (xy 331.47 -5.08))
+  (wire (pts (xy 330.2 -3.81) (xy 330.2 -5.08))
     (stroke (width 0) (type default))
   )
@@
     (stroke (width 0) (type default))
   )
-  (wire (pts (xy 337.82 -5.08) (xy 349.25 -5.08))
-    (stroke (width 0) (type default))
-  )
   (wire (pts (xy 259.08 63.5) (xy 259.08 60.96))
     (stroke (width 0) (type default))
@@
     (stroke (width 0) (type default))
   )
+  (wire (pts (xy 342.9 -5.08) (xy 342.9 -3.81))
+    (stroke (width 0) (type default))
+  )
   (wire (pts (xy 381 30.48) (xy 377.19 30.48))
     (stroke (width 0) (type default))
@@
     (stroke (width 0) (type default))
   )
-  (wire (pts (xy 337.82 -5.08) (xy 331.47 -5.08))
+  (wire (pts (xy 336.55 -5.08) (xy 342.9 -5.08))
     (stroke (width 0) (type default))
   )
@@
     (stroke (width 0) (type default))
   )
+  (wire (pts (xy 336.55 -5.08) (xy 330.2 -5.08))
+    (stroke (width 0) (type default))
+  )
+  (wire (pts (xy 342.9 3.81) (xy 342.9 5.08))
+    (stroke (width 0) (type default))
+  )
   (polyline (pts (xy 142.24 54.61) (xy 142.24 54.61))
     (stroke (width 0) (type default))
@@
     (stroke (width 0) (type default))
   )
-  (wire (pts (xy 331.47 3.81) (xy 331.47 5.08))
+  (wire (pts (xy 330.2 3.81) (xy 330.2 5.08))
     (stroke (width 0) (type default))
   )
@@
     (stroke (width 0) (type default))
   )
-  (wire (pts (xy 337.82 3.81) (xy 337.82 5.08))
+  (wire (pts (xy 336.55 3.81) (xy 336.55 5.08))
     (stroke (width 0) (type default))
   )
@@
     (stroke (width 0) (type default))
   )
+  (wire (pts (xy 342.9 -5.08) (xy 349.25 -5.08))
+    (stroke (width 0) (type default))
+  )
   (wire (pts (xy 486.41 91.44) (xy 486.41 90.17))
     (stroke (width 0) (type default))
@@
     (stroke (width 0) (type default))
   )
-  (wire (pts (xy 337.82 -5.08) (xy 337.82 -3.81))
+  (wire (pts (xy 336.55 -5.08) (xy 336.55 -3.81))
     (stroke (width 0) (type default))
   )
@@
     )
   )
+  (symbol (lib_id "Device:C") (at 342.9 0 0) (unit 1)
+    (in_bom yes) (on_board yes) (dnp no)
+    (property "Reference" "C11" (at 345.821 -1.1684 0)
+      (effects (font (size 1.27 1.27)) (justify left))
+    )
+    (property "Value" "0.1uF" (at 345.821 1.143 0)
+      (effects (font (size 1.27 1.27)) (justify left))
+    )
+    (property "Footprint" "Capacitor_SMD:C_0805_2012Metric" (at 343.8652 3.81 0)
+      (effects (font (size 1.27 1.27)) hide)
+    )
+    (property "Datasheet" "~" (at 342.9 0 0)
+      (effects (font (size 1.27 1.27)) hide)
+    )
+    (property "Digi-Key_PN" "311-1344-1-ND" (at 342.9 0 0)
+      (effects (font (size 1.27 1.27)) hide)
+    )
+    (pin "1")
+    (pin "2")
+    (instances
+      (project "rpi-pico-debugger-shoe"
+        (path "/be7be351-63b7-49f6-8c40-c4ef86885582"
+          (reference "C11") (unit 1)
+        )
+      )
+      (project "PD-LabSupply"
+        (path "/e63e39d7-6ac0-4ffd-8aa3-1841a4541b55"
+          (reference "C31") (unit 1)
+        )
+      )
+    )
+  )
   (symbol (lib_id "power:VDD") (at 93.98 101.6 0) (unit 1)
     (in_bom yes) (on_board yes) (dnp no)
@@
     )
   )
-  (symbol (lib_id "Device:C") (at 337.82 0 0) (unit 1)
+  (symbol (lib_id "Device:C") (at 336.55 0 0) (unit 1)
     (in_bom yes) (on_board yes) (dnp no)
-    (property "Reference" "C11" (at 340.741 -1.1684 0)
+    (property "Reference" "C11" (at 335.28 -8.89 0)
       (effects (font (size 1.27 1.27)) (justify left))
     )
-    (property "Value" "0.1uF" (at 340.741 1.143 0)
+    (property "Value" "1uF 50v" (at 332.74 -6.35 0)
       (effects (font (size 1.27 1.27)) (justify left))
     )
-    (property "Footprint" "Capacitor_SMD:C_0805_2012Metric" (at 338.7852 3.81 0)
+    (property "Footprint" "Capacitor_SMD:C_0805_2012Metric" (at 337.5152 3.81 0)
       (effects (font (size 1.27 1.27)) hide)
     )
-    (property "Datasheet" "~" (at 337.82 0 0)
+    (property "Datasheet" "~" (at 336.55 0 0)
       (effects (font (size 1.27 1.27)) hide)
     )
-    (property "Digi-Key_PN" "311-1344-1-ND" (at 337.82 0 0)
+    (property "Digi-Key_PN" "311-1344-1-ND" (at 336.55 0 0)
       (effects (font (size 1.27 1.27)) hide)
     )
@@
     )
   )
+  (symbol (lib_id "power:GND") (at 342.9 5.08 0) (unit 1)
+    (in_bom yes) (on_board yes) (dnp no)
+    (property "Reference" "#PWR0128" (at 342.9 11.43 0)
+      (effects (font (size 1.27 1.27)) hide)
+    )
+    (property "Value" "GND" (at 343.027 9.4742 0)
+      (effects (font (size 1.27 1.27)))
+    )
+    (property "Footprint" "" (at 342.9 5.08 0)
+      (effects (font (size 1.27 1.27)) hide)
+    )
+    (property "Datasheet" "" (at 342.9 5.08 0)
+      (effects (font (size 1.27 1.27)) hide)
+    )
+    (pin "1")
+    (instances
+      (project "rpi-pico-debugger-shoe"
+        (path "/be7be351-63b7-49f6-8c40-c4ef86885582"
+          (reference "#PWR0128") (unit 1)
+        )
+      )
+      (project "PD-LabSupply"
+        (path "/e63e39d7-6ac0-4ffd-8aa3-1841a4541b55"
+          (reference "#PWR061") (unit 1)
+        )
+      )
+    )
+  )
   (symbol (lib_id "-Passive:C") (at 123.19 147.32 0) (unit 1)
     (in_bom yes) (on_board yes) (dnp no)
@@
     )
   )
-  (symbol (lib_id "power:GND") (at 337.82 5.08 0) (unit 1)
+  (symbol (lib_id "power:GND") (at 336.55 5.08 0) (unit 1)
     (in_bom yes) (on_board yes) (dnp no)
-    (property "Reference" "#PWR0128" (at 337.82 11.43 0)
+    (property "Reference" "#PWR0128" (at 336.55 11.43 0)
       (effects (font (size 1.27 1.27)) hide)
     )
-    (property "Value" "GND" (at 337.947 9.4742 0)
+    (property "Value" "GND" (at 336.677 9.4742 0)
       (effects (font (size 1.27 1.27)))
     )
-    (property "Footprint" "" (at 337.82 5.08 0)
+    (property "Footprint" "" (at 336.55 5.08 0)
       (effects (font (size 1.27 1.27)) hide)
     )
-    (property "Datasheet" "" (at 337.82 5.08 0)
+    (property "Datasheet" "" (at 336.55 5.08 0)
       (effects (font (size 1.27 1.27)) hide)
     )
@@
     )
   )
-  (symbol (lib_id "Device:C") (at 331.47 0 0) (unit 1)
+  (symbol (lib_id "Device:C") (at 330.2 0 0) (unit 1)
     (in_bom yes) (on_board yes) (dnp no)
-    (property "Reference" "C9" (at 323.85 -1.0414 0)
+    (property "Reference" "C9" (at 322.58 -1.0414 0)
       (effects (font (size 1.27 1.27)) (justify left))
     )
-    (property "Value" "0.1uF" (at 323.85 1.27 0)
+    (property "Value" "0.1uF" (at 322.58 1.27 0)
       (effects (font (size 1.27 1.27)) (justify left))
     )
-    (property "Footprint" "Capacitor_SMD:C_0805_2012Metric" (at 332.4352 3.81 0)
+    (property "Footprint" "Capacitor_SMD:C_0805_2012Metric" (at 331.1652 3.81 0)
       (effects (font (size 1.27 1.27)) hide)
     )
-    (property "Datasheet" "~" (at 331.47 0 0)
+    (property "Datasheet" "~" (at 330.2 0 0)
       (effects (font (size 1.27 1.27)) hide)
     )
-    (property "Digi-Key_PN" "311-1344-1-ND" (at 331.47 0 0)
+    (property "Digi-Key_PN" "311-1344-1-ND" (at 330.2 0 0)
       (effects (font (size 1.27 1.27)) hide)
     )
@@
     )
   )
-  (symbol (lib_id "power:GND") (at 331.47 5.08 0) (unit 1)
+  (symbol (lib_id "power:GND") (at 330.2 5.08 0) (unit 1)
     (in_bom yes) (on_board yes) (dnp no)
-    (property "Reference" "#PWR0129" (at 331.47 11.43 0)
+    (property "Reference" "#PWR0129" (at 330.2 11.43 0)
       (effects (font (size 1.27 1.27)) hide)
     )
-    (property "Value" "GND" (at 331.597 9.4742 0)
+    (property "Value" "GND" (at 330.327 9.4742 0)
       (effects (font (size 1.27 1.27)))
     )
-    (property "Footprint" "" (at 331.47 5.08 0)
+    (property "Footprint" "" (at 330.2 5.08 0)
       (effects (font (size 1.27 1.27)) hide)
     )
-    (property "Datasheet" "" (at 331.47 5.08 0)
+    (property "Datasheet" "" (at 330.2 5.08 0)
       (effects (font (size 1.27 1.27)) hide)
     )

Commit message: layout finished
Parts:
- removed J2, J4, J5: Conn_01x02, Connector_PinHeader_2.54mm:PinHeader_1x02_P2.54mm_Vertical, symbol -Connector:Conn_01x02
- removed J7: Conn_01x02, Connector_PinHeader_2.54mm:PinHeader_1x02_P2.54mm_Horizontal, symbol -Connector:Conn_01x02
- added Y1: Crystal_GND24, symbol Device:Crystal_GND24
Connections:
- net +5V: now also J8.3 (Pin_3)
- net GND: now also J8.1 (Pin_1)
- net SCL: now also J8.4 (Pin_4)
- net SDA: now also J8.2 (Pin_2)
Other:
- moved on the sheet: J8

Commit message: save
Parts:
- removed J8: Conn_02x02_Counter_Clockwise, Connector_PinSocket_2.54mm:PinSocket_2x02_P2.54mm_Horizontal, symbol Connector_Generic:Conn_02x02_Counter_Clockwise
- removed XTAL1: ABLS-12.000MHZ-B2-T, ABLS_12_000MHZ_B2_T:XTAL_HC&slash_49US_ABLS_ABR, symbol ABLS_12_000MHZ_B2_T:ABLS-12.000MHZ-B2-T
- added J2: Conn_02x02_Odd_Even, symbol Connector_Generic:Conn_02x02_Odd_Even
- C13, C15: value 27pF -> 15pF
- Y1: footprint (none) -> Crystal:Crystal_SMD_3225-4Pin_3.2x2.5mm
Connections:
- net +5V: now also J2.3 (Pin_3)
- net GND: now also Y1.2, Y1.4, J2.1 (Pin_1)
- net SCL: now also J2.4 (Pin_4)
- net SDA: now also J2.2 (Pin_2)
- net XIN: now also Y1.1
- net at C15.1, R7.2: now also Y1.3
Other:
- moved on the sheet: Y1
