File: PD-LabSupply.kicad_sch (KiCad schematic)
At the start: 85 parts, among them J1 Conn_01x02, J2 Conn_02x02_Odd_Even, J3 USB_C_Receptacle_USB2.0, J6 Conn_01x07, Q1 BC847, Q4 IRF9393, SW1 SW_DIP_x06, SW2 SW_DPST_x2, SW3 SW_Push, SW4 SW_Push, SW5 SW_DPST_x2, SW6 SW_Push, U1 SRV05-4, U3 TMCS1108, U4 AP33772, U5 RP2040, U6 oledSym, U7 LMR54410, U8 AP2112K-3.3TRG1, U9 W25Q16JVSSIQ, Y1 Crystal_GND24

Commit message: save
Parts:
- added SW7: SW_Push, Button_Switch_SMD:SW_SPST_PTS810, symbol Switch:SW_Push
- J2: footprint (none) -> Connector_PinSocket_2.54mm:PinSocket_2x02_P2.54mm_Horizontal
- L1: footprint -Passive:L_4012 -> Inductor_SMD:L_Coilcraft_XAL5050-XXX
- SW3, SW4, SW6: footprint Button_Switch_SMD:SW_SPST_TL3305B -> Button_Switch_SMD:SW_SPST_PTS810
Connections:
- net GND: now also SW7.1
- net BTN_SEL: now reaches U5.27 (GPIO16)
- net BTN_SEL: now also SW7.2
Changed lines of the file:
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@@
   (junction (at 87.63 60.96) (diameter 0) (color 0 0 0 0)
   )
+  (junction (at 26.67 135.89) (diameter 0) (color 0 0 0 0)
+  )
   (junction (at 121.92 72.39) (diameter 0) (color 0 0 0 0)
   )
@@
     (stroke (width 0) (type default))
   )
+  (wire (pts (xy 377.19 55.88) (xy 381 55.88))
+    (stroke (width 0) (type default))
+  )
   (polyline (pts (xy 107.95 162.56) (xy 161.29 162.56))
     (stroke (width 0) (type default))
@@
     (stroke (width 0) (type default))
   )
+  (wire (pts (xy 26.67 135.89) (xy 26.67 138.43))
+    (stroke (width 0) (type default))
+  )
   (wire (pts (xy 405.13 132.08) (xy 405.13 133.35))
     (stroke (width 0) (type default))
@@
     (stroke (width 0) (type default))
   )
-  (wire (pts (xy 26.67 129.54) (xy 26.67 133.35))
+  (wire (pts (xy 26.67 129.54) (xy 26.67 135.89))
     (stroke (width 0) (type default))
   )
@@
     (stroke (width 0) (type default))
   )
+  (wire (pts (xy 26.67 135.89) (xy 29.21 135.89))
+    (stroke (width 0) (type default))
+  )
   (wire (pts (xy 130.81 124.46) (xy 133.35 124.46))
     (stroke (width 0) (type default))
@@
     (stroke (width 0) (type default))
   )
+  (wire (pts (xy 39.37 135.89) (xy 40.64 135.89))
+    (stroke (width 0) (type default))
+  )
   (wire (pts (xy 381 43.18) (xy 377.19 43.18))
     (stroke (width 0) (type default))
@@
     )
   )
+  (global_label "BTN_SEL" (shape input) (at 381 55.88 0) (fields_autoplaced)
+    (effects (font (size 1.27 1.27)) (justify left))
+    (property "Intersheetrefs" "${INTERSHEET_REFS}" (at 391.2533 55.88 0)
+      (effects (font (size 1.27 1.27)) (justify left) hide)
+    )
+  )
   (global_label "XIN" (shape input) (at 323.85 60.96 180) (fields_autoplaced)
     (effects (font (size 1.27 1.27)) (justify right))
@@
     )
   )
+  (global_label "BTN_SEL" (shape input) (at 40.64 135.89 0) (fields_autoplaced)
+    (effects (font (size 1.27 1.27)) (justify left))
+    (property "Intersheetrefs" "${INTERSHEET_REFS}" (at 50.8933 135.89 0)
+      (effects (font (size 1.27 1.27)) (justify left) hide)
+    )
+  )
   (global_label "ENOUT" (shape input) (at 218.44 134.62 0) (fields_autoplaced)
     (effects (font (size 1.27 1.27)) (justify left))
@@
       (effects (font (size 1.27 1.27)))
     )
-    (property "Footprint" "-Passive:L_4012" (at 115.57 64.77 0)
+    (property "Footprint" "Inductor_SMD:L_Coilcraft_XAL5050-XXX" (at 115.57 64.77 0)
       (effects (font (size 1.27 1.27)) hide)
     )
@@
       (effects (font (size 1.27 1.27)))
     )
-    (property "Footprint" "Button_Switch_SMD:SW_SPST_TL3305B" (at 419.1 82.55 0)
+    (property "Footprint" "Button_Switch_SMD:SW_SPST_PTS810" (at 419.1 82.55 0)
       (effects (font (size 1.27 1.27)) hide)
     )
@@
   (symbol (lib_id "Switch:SW_Push") (at 34.29 129.54 0) (unit 1)
     (in_bom yes) (on_board yes) (dnp no)
-    (property "Reference" "SW3" (at 35.56 135.89 0)
+    (property "Reference" "SW3" (at 22.86 132.08 0)
       (effects (font (size 1.27 1.27)))
     )
-    (property "Value" "SW_Push" (at 34.29 132.08 0)
+    (property "Value" "SW_Push" (at 21.59 128.27 0)
       (effects (font (size 1.27 1.27)))
     )
-    (property "Footprint" "Button_Switch_SMD:SW_SPST_TL3305B" (at 34.29 124.46 0)
+    (property "Footprint" "Button_Switch_SMD:SW_SPST_PTS810" (at 34.29 124.46 0)
       (effects (font (size 1.27 1.27)) hide)
     )
@@
     )
   )
+  (symbol (lib_id "Switch:SW_Push") (at 34.29 135.89 0) (unit 1)
+    (in_bom yes) (on_board yes) (dnp no)
+    (property "Reference" "SW7" (at 35.56 142.24 0)
+      (effects (font (size 1.27 1.27)))
+    )
+    (property "Value" "SW_Push" (at 34.29 138.43 0)
+      (effects (font (size 1.27 1.27)))
+    )
+    (property "Footprint" "Button_Switch_SMD:SW_SPST_PTS810" (at 34.29 130.81 0)
+      (effects (font (size 1.27 1.27)) hide)
+    )
+    (property "Datasheet" "~" (at 34.29 130.81 0)
+      (effects (font (size 1.27 1.27)) hide)
+    )
+    (pin "1")
+    (pin "2")
+    (instances
+      (project "PD-LabSupply"
+        (path "/e63e39d7-6ac0-4ffd-8aa3-1841a4541b55"
+          (reference "SW7") (unit 1)
+        )
+      )
+    )
+  )
   (symbol (lib_id "Device:Thermistor") (at 135.89 140.97 0) (unit 1)
     (in_bom yes) (on_board yes) (dnp no)
@@
       (effects (font (size 1.27 1.27)))
     )
-    (property "Footprint" "Button_Switch_SMD:SW_SPST_TL3305B" (at 33.02 119.38 0)
+    (property "Footprint" "Button_Switch_SMD:SW_SPST_PTS810" (at 33.02 119.38 0)
       (effects (font (size 1.27 1.27)) hide)
     )
@@
       (effects (font (size 1.27 1.27)))
     )
-    (property "Footprint" "" (at 351.79 138.43 0)
+    (property "Footprint" "Connector_PinSocket_2.54mm:PinSocket_2x02_P2.54mm_Horizontal" (at 351.79 138.43 0)
       (effects (font (size 1.27 1.27)) hide)
     )
@@
     )
   )
-  (symbol (lib_id "-Flag:GND") (at 26.67 133.35 0) (unit 1)
+  (symbol (lib_id "-Flag:GND") (at 26.67 138.43 0) (unit 1)
     (in_bom yes) (on_board yes) (dnp no) (fields_autoplaced)
-    (property "Reference" "#PWR0116" (at 26.67 139.7 0)
+    (property "Reference" "#PWR0116" (at 26.67 144.78 0)
       (effects (font (size 1.27 1.27)) hide)
     )
-    (property "Value" "GND" (at 26.67 138.43 0)
+    (property "Value" "GND" (at 26.67 143.51 0)
       (effects (font (size 1.27 1.27)))
     )
-    (property "Footprint" "" (at 26.67 133.35 0)
+    (property "Footprint" "" (at 26.67 138.43 0)
       (effects (font (size 1.27 1.27)) hide)
     )
-    (property "Datasheet" "" (at 26.67 133.35 0)
+    (property "Datasheet" "" (at 26.67 138.43 0)
       (effects (font (size 1.27 1.27)) hide)
     )
