File: PD-LabSupply.kicad_sch (KiCad schematic)
At the start: 86 parts, among them J1 Conn_01x02, J2 Conn_02x02_Odd_Even, J3 USB_C_Receptacle_USB2.0, J6 Conn_01x07, Q1 BC847, Q4 IRF9393, SW1 SW_DIP_x06, SW2 SW_DPST_x2, SW3 SW_Push, SW4 SW_Push, SW5 SW_DPST_x2, SW6 SW_Push, SW7 SW_Push, U1 SRV05-4, U3 TMCS1108, U4 AP33772, U5 RP2040, U6 oledSym, U7 LMR54410, U8 AP2112K-3.3TRG1, U9 W25Q16JVSSIQ, Y1 Crystal_GND24

Commit message: fertig
Parts:
- removed J3: USB_C_Receptacle_USB2.0, Connector_USB:USB_C_Receptacle_JAE_DX07S016JA1R1500, symbol Connector:USB_C_Receptacle_USB2.0
- added J4: USB4500-03-0-A, USB4500_03_0_A:CONN_USB4500_GCT, symbol USB4500_03_0_A:USB4500-03-0-A
Connections:
- net CC1: now also J4.B5 (CC2)
- net CC2: now also J4.A5 (CC1)
- net D_N: now also J4.A7 (DN1), J4.B7 (DN2)
- net D_P: now also J4.A6 (DP1), J4.B6 (DP2)
- net GND: now also J4.A1 (GND), J4.A12 (GND), J4.B1 (GND), J4.B12 (GND)
- net VDD: now also J4.A4 (VBUS), J4.A9 (VBUS), J4.B4 (VBUS), J4.B9 (VBUS)
Other:
- moved on the sheet: C12

Commit message: save
Parts:
- removed Q1: BC847, Package_TO_SOT_SMD:SOT-23, symbol PCM_Transistor_BJT_AKL:BC847
- removed Q4: IRF9393, Package_SO:SOIC-8_3.9x4.9mm_P1.27mm, symbol IRF9393:IRF9393
- removed R5, R7: 5k1, Resistor_SMD:R_0805_2012Metric, symbol -Passive:R
- removed R6: 10k, Resistor_SMD:R_0805_2012Metric, symbol -Passive:R
- removed R8: 1k, Resistor_SMD:R_0805_2012Metric, symbol -Passive:R
- added Q2: DMN3008SFGQ-7, DMN3008SFGQ-7:DMG7401SFG13, symbol DMN3008SFGQ-7:DMN3008SFGQ-7
- renumbered SW5 to SW2, SW2 to SW5
Connections:
- net BTN_DOWN: now also U5.29 (GPIO18); no longer U5.17 (GPIO14)
- net BTN_SEL: now also U5.30 (GPIO19); no longer U5.27 (GPIO16)
- net BTN_UP: now also U5.31 (GPIO20); no longer U5.18 (GPIO15)
- net ENOUT: now also U4.23 (PWR_EN), Q2.4 (G); no longer U5.32 (GPIO21)
- net HALL_IN: now also Q2.5 (D_1), Q2.6 (D_2), Q2.7 (D_3), Q2.8 (D_4)
- net LED: now also U5.35 (GPIO23); no longer U5.5 (GPIO3)
- net SW_OUT: now also U5.34 (GPIO22); no longer U5.15 (GPIO12)
- net SW_VA: now also U5.32 (GPIO21); no longer U5.16 (GPIO13)
- net VBUS: now also Q2.1 (S_1), Q2.2 (S_2), Q2.3 (S_3)
Other:
- moved on the sheet: C2, C4, C6, C7

Commit message: finished
Parts:
- removed H1, H3: MountingHole, MountingHole:MountingHole_2.5mm, symbol -Connector:MountingHole
- removed J4: USB4500-03-0-A, USB4500_03_0_A:CONN_USB4500_GCT, symbol USB4500_03_0_A:USB4500-03-0-A
- removed SW2, SW5: SW_DPST_x2, Button_Switch_SMD:SW_SPDT_PCM12, symbol Switch:SW_DPST_x2
- added J3: USB4520-03-0-A, USB4520_03_0_A:CONN12_USB4520-03-0-A_GCT, symbol USB4520_03_0_A:USB4520-03-0-A
- added SW2, SW8: JS202011JAQN, JS202011JAQN:JS202011JAQN, symbol JS202011JAQN:JS202011JAQN
- L1: footprint Inductor_SMD:L_Coilcraft_XAL5050-XXX -> Inductor_SMD:L_Taiyo-Yuden_MD-5050
- U3: footprint Package_SO:SOIC-8_3.9x4.9mm_P1.27mm -> PCM_4ms_Package_SOIC:SOIC-8_3.9x4.9mm_Pitch1.27mm
- U4: footprint Package_DFN_QFN:WQFN-24-1EP_4x4mm_P0.5mm_EP2.6x2.6mm_ThermalVias -> AP33772:AP33772
- U8: footprint Package_TO_SOT_SMD:SOT-23-5 -> AP2112K_3_3TRG1:SOT_RG1_DIO
Connections:
- net ADC0: now also U5.41 (GPIO29_ADC3); no longer U5.38 (GPIO26_ADC0)
- net CC1: now also J3.CC1
- net CC2: now also J3.CC2
- net D_N: now also J3.D_N (D-)
- net D_P: now also J3.D_P (D+)
- net ENOUT: now also Q2.G; no longer J6.2 (Pin_2), Q2.4 (G)
- net GND: now also J3.GND, SW2.3, SW8.3
- net HALL_IN: now also Q2.D; no longer Q2.5 (D_1), Q2.6 (D_2), Q2.7 (D_3), Q2.8 (D_4)
- net LED: now also U5.34 (GPIO22); no longer U5.35 (GPIO23)
- net SW_OUT: now also U5.35 (GPIO23), SW8.1, SW8.2; no longer U5.34 (GPIO22)
- net SW_VA: now also SW2.1, SW2.2
- net VBUS: now also Q2.S; no longer Q2.1 (S_1), Q2.2 (S_2), Q2.3 (S_3)
- net VDD: now also J3.VBUS
- net EXT_OUT: now reaches U5.15 (GPIO12)
- net EXT_OUT: now also J6.2 (Pin_2)
- net SHIELD: no longer names the net of C1.1, R1.1
- net SHIELD: now also J3.SHIELD
- no-connect marks 4 -> 8
Other:
- moved on the sheet: C1, C12, C7, R1

Commit message: bestellung
Other:
- title: PD-LabSupply -> PD-LabSupply_Core-Module
Changed lines of the file:
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@@
   (paper "A4")
   (title_block
-    (title "PD-LabSupply")
-    (date "2023-11-26")
-    (rev "3.1")
+    (title "PD-LabSupply_Core-Module")
+    (date "2023-12-11")
+    (rev "4.2")
     (company "HTL Rankweil")
     (comment 1 "Johannes Melcher-Millner")

Commit message: changes
Parts:
- added R5: 1k, Resistor_SMD:R_0805_2012Metric, symbol -Passive:R
Connections:
- net ENOUT: now also R5.1; no longer Q2.G
- new net: Q2.G, R5.2
Other:
- moved on the sheet: C7, Q2
Changed lines of the file:
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@@
   (junction (at 25.4 92.71) (diameter 0) (color 0 0 0 0)
   )
-  (junction (at 203.2 140.97) (diameter 0) (color 0 0 0 0)
+  (junction (at 217.17 140.97) (diameter 0) (color 0 0 0 0)
   )
   (junction (at 133.35 124.46) (diameter 0) (color 0 0 0 0)
@@
     (stroke (width 0) (type default))
   )
+  (wire (pts (xy 199.39 133.35) (xy 201.93 133.35))
+    (stroke (width 0) (type default))
+  )
   (wire (pts (xy 93.98 121.92) (xy 93.98 109.22))
     (stroke (width 0) (type default))
@@
     (stroke (width 0) (type default))
   )
-  (wire (pts (xy 203.2 148.59) (xy 203.2 147.32))
+  (wire (pts (xy 217.17 148.59) (xy 217.17 147.32))
     (stroke (width 0) (type default))
   )
@@
     (stroke (width 0) (type default))
   )
-  (wire (pts (xy 203.2 140.97) (xy 203.2 139.7))
+  (wire (pts (xy 217.17 140.97) (xy 217.17 139.7))
     (stroke (width 0) (type default))
   )
@@
     (stroke (width 0) (type default))
   )
-  (wire (pts (xy 198.12 133.35) (xy 196.85 133.35))
+  (wire (pts (xy 212.09 133.35) (xy 209.55 133.35))
     (stroke (width 0) (type default))
   )
@@
     (stroke (width 0) (type default))
   )
-  (wire (pts (xy 203.2 140.97) (xy 203.2 142.24))
+  (wire (pts (xy 217.17 140.97) (xy 217.17 142.24))
     (stroke (width 0) (type default))
   )
@@
     (stroke (width 0) (type default))
   )
-  (wire (pts (xy 203.2 125.73) (xy 203.2 127))
+  (wire (pts (xy 217.17 125.73) (xy 217.17 127))
     (stroke (width 0) (type default))
   )
@@
     (stroke (width 0) (type default))
   )
-  (wire (pts (xy 203.2 140.97) (xy 205.74 140.97))
+  (wire (pts (xy 217.17 140.97) (xy 219.71 140.97))
     (stroke (width 0) (type default))
   )
@@
     (stroke (width 0) (type default))
   )
-  (wire (pts (xy 185.42 125.73) (xy 203.2 125.73))
+  (wire (pts (xy 185.42 125.73) (xy 217.17 125.73))
     (stroke (width 0) (type default))
   )
@@
     )
   )
-  (global_label "ENOUT" (shape input) (at 196.85 133.35 180) (fields_autoplaced)
+  (global_label "ENOUT" (shape input) (at 199.39 133.35 180) (fields_autoplaced)
     (effects (font (size 1.27 1.27)) (justify right))
-    (property "Intersheetrefs" "${INTERSHEET_REFS}" (at 188.4109 133.35 0)
+    (property "Intersheetrefs" "${INTERSHEET_REFS}" (at 190.9509 133.35 0)
       (effects (font (size 1.27 1.27)) (justify right) hide)
     )
@@
     )
   )
-  (global_label "HALL_IN" (shape input) (at 205.74 140.97 0) (fields_autoplaced)
+  (global_label "HALL_IN" (shape input) (at 219.71 140.97 0) (fields_autoplaced)
     (effects (font (size 1.27 1.27)) (justify left))
-    (property "Intersheetrefs" "${INTERSHEET_REFS}" (at 215.4492 140.97 0)
+    (property "Intersheetrefs" "${INTERSHEET_REFS}" (at 229.4192 140.97 0)
       (effects (font (size 1.27 1.27)) (justify left) hide)
     )
@@
     )
   )
-  (symbol (lib_id "-Flag:GND") (at 203.2 148.59 0) (unit 1)
+  (symbol (lib_id "-Flag:GND") (at 217.17 148.59 0) (unit 1)
     (in_bom yes) (on_board yes) (dnp no)
-    (property "Reference" "#PWR09" (at 203.2 154.94 0)
+    (property "Reference" "#PWR09" (at 217.17 154.94 0)
       (effects (font (size 1.27 1.27)) hide)
     )
-    (property "Value" "GND" (at 207.01 151.13 0)
+    (property "Value" "GND" (at 220.98 151.13 0)
       (effects (font (size 1.016 1.016)))
     )
-    (property "Footprint" "" (at 203.2 148.59 0)
+    (property "Footprint" "" (at 217.17 148.59 0)
       (effects (font (size 1.27 1.27)) hide)
     )
-    (property "Datasheet" "" (at 203.2 148.59 0)
+    (property "Datasheet" "" (at 217.17 148.59 0)
       (effects (font (size 1.27 1.27)) hide)
     )
@@
     )
   )
-  (symbol (lib_id "-Passive:C") (at 203.2 144.78 0) (unit 1)
+  (symbol (lib_id "-Passive:C") (at 217.17 144.78 0) (unit 1)
     (in_bom yes) (on_board yes) (dnp no)
-    (property "Reference" "C7" (at 207.01 144.78 0)
+    (property "Reference" "C7" (at 220.98 144.78 0)
       (effects (font (size 1.27 1.27)) (justify left))
     )
-    (property "Value" "1uF 50V" (at 205.74 147.32 0)
+    (property "Value" "1uF 50V" (at 219.71 147.32 0)
       (effects (font (size 1.016 1.016)) (justify left))
     )
-    (property "Footprint" "Capacitor_SMD:C_0805_2012Metric" (at 204.1652 148.59 0)
+    (property "Footprint" "Capacitor_SMD:C_0805_2012Metric" (at 218.1352 148.59 0)
       (effects (font (size 1.27 1.27)) hide)
     )
-    (property "Datasheet" "~" (at 203.2 144.78 0)
+    (property "Datasheet" "~" (at 217.17 144.78 0)
       (effects (font (size 1.27 1.27)) hide)
     )
@@
     )
   )
-  (symbol (lib_id "DMN3008SFGQ-7:DMN3008SFGQ-7") (at 200.66 142.24 0) (unit 1)
+  (symbol (lib_id "DMN3008SFGQ-7:DMN3008SFGQ-7") (at 214.63 142.24 0) (unit 1)
     (in_bom yes) (on_board yes) (dnp no)
-    (property "Reference" "Q2" (at 214.63 133.35 0)
+    (property "Reference" "Q2" (at 228.6 133.35 0)
       (effects (font (size 1.27 1.27)))
     )
-    (property "Value" "DMN3008SFGQ-7" (at 214.63 135.89 0)
+    (property "Value" "DMN3008SFGQ-7" (at 228.6 135.89 0)
       (effects (font (size 1.27 1.27)))
     )
-    (property "Footprint" "DMN3008SFGQ-7:DMG7401SFG13" (at 222.25 237.16 0)
+    (property "Footprint" "DMN3008SFGQ-7:DMG7401SFG13" (at 236.22 237.16 0)
       (effects (font (size 1.27 1.27)) (justify left top) hide)
     )
-    (property "Datasheet" "https://www.diodes.com/assets/Datasheets/DMN3008SFGQ.pdf" (at 222.25 337.16 0)
+    (property "Datasheet" "https://www.diodes.com/assets/Datasheets/DMN3008SFGQ.pdf" (at 236.22 337.16 0)
       (effects (font (size 1.27 1.27)) (justify left top) hide)
     )
-    (property "Height" "" (at 222.25 537.16 0)
+    (property "Height" "" (at 236.22 537.16 0)
       (effects (font (size 1.27 1.27)) (justify left top) hide)
     )
-    (property "Mouser Part Number" "621-DMN3008SFGQ-7" (at 222.25 637.16 0)
+    (property "Mouser Part Number" "621-DMN3008SFGQ-7" (at 236.22 637.16 0)
       (effects (font (size 1.27 1.27)) (justify left top) hide)
     )
-    (property "Mouser Price/Stock" "https://www.mouser.co.uk/ProductDetail/Diodes-Incorporated/DMN3008SFGQ-7?qs=4EhzHfbM1GgrzSOUtnha%2FQ%3D%3D" (at 222.25 737.16 0)
+    (property "Mouser Price/Stock" "https://www.mouser.co.uk/ProductDetail/Diodes-Incorporated/DMN3008SFGQ-7?qs=4EhzHfbM1GgrzSOUtnha%2FQ%3D%3D" (at 236.22 737.16 0)
       (effects (font (size 1.27 1.27)) (justify left top) hide)
     )
-    (property "Manufacturer_Name" "Diodes Incorporated" (at 222.25 837.16 0)
+    (property "Manufacturer_Name" "Diodes Incorporated" (at 236.22 837.16 0)
       (effects (font (size 1.27 1.27)) (justify left top) hide)
     )
-    (property "Manufacturer_Part_Number" "DMN3008SFGQ-7" (at 222.25 937.16 0)
+    (property "Manufacturer_Part_Number" "DMN3008SFGQ-7" (at 236.22 937.16 0)
       (effects (font (size 1.27 1.27)) (justify left top) hide)
     )
@@
         )
       )
+    )
+  )
+  (symbol (lib_id "-Passive:R") (at 205.74 133.35 90) (unit 1)
+    (in_bom yes) (on_board yes) (dnp no)
+    (property "Reference" "R5" (at 204.47 138.43 0)
+      (effects (font (size 1.27 1.27)) (justify left))
+    )
+    (property "Value" "1k" (at 208.28 138.43 0)
+      (effects (font (size 1.016 1.016)) (justify left))
+    )
+    (property "Footprint" "Resistor_SMD:R_0805_2012Metric" (at 205.994 132.334 90)
+      (effects (font (size 1.27 1.27)) hide)
+    )
+    (property "Datasheet" "" (at 205.74 133.35 0)
+      (effects (font (size 1.27 1.27)) hide)
+    )
+    (pin "1")
+    (pin "2")
+    (instances
+      (project "PD-LabSupply"
+        (path "/e63e39d7-6ac0-4ffd-8aa3-1841a4541b55"
+          (reference "R5") (unit 1)
+        )
+      )

Commit message: finished
Parts:
- removed J6: Conn_01x07, Connector_PinSocket_2.54mm:PinSocket_1x07_P2.54mm_Vertical_SMD_Pin1Left, symbol Connector_Generic:Conn_01x07
- added R6, R7: X, Resistor_SMD:R_0805_2012Metric, symbol -Passive:R
- added TP10, TP11, TP12, TP13, TP7, TP8, TP9: TestPoint, TestPoint:TestPoint_Pad_D1.5mm, symbol -Connector:TestPoint
- C11, C16, C28, C29, C8: value 1uF 50v -> 1uF 50V
- C13, C15: value 15pF -> 18pF
- C9: value 22u 50V -> 22uF 50V
- TP1, TP2, TP3, TP4: footprint TestPoint:TestPoint_Pad_D2.0mm -> TestPoint:TestPoint_Pad_D1.5mm
Connections:
- net EN12V: now also TP11.1
- net EN15V: now also TP10.1
- net EN20V: now also TP9.1
- net EN5V: now also TP13.1
- net EN9V: now also TP12.1
- net EXT_OUT: now also TP8.1
- net GND: now also R7.2, TP7.1
- net HALL_IN: now also Q2.S; no longer Q2.D
- net VBUS: now also Q2.D, R6.1; no longer Q2.S
- net HALL_ADC: now reaches U5.40 (GPIO28_ADC2)
- net HALL_ADC: now also U3.7 (VOUT)
- net ADC0 renamed V_ADC
- net V_ADC: now also R6.2, R7.1; no longer U3.7 (VOUT)
- no-connect marks 8 -> 19
Other:
- moved on the sheet: C11, H2, H4, U3
